File: Computer/Computer.sch (KiCad schematic (older format))
At the start: 0 parts

Commit message: computer changes
Changed lines of the file:
@@
 LIBS:contrib
 LIBS:valves
+LIBS:Computer-cache
 EELAYER 25 0
 EELAYER END
 $Descr A4 11693 8268
 encoding utf-8
-Sheet 1 2
+Sheet 1 4
 Title ""
 Date ""
@@
 F1 "ALU.sch" 60
 $EndSheet
+$Sheet
+S -4300 -1600 3850 2800
+U 5A218830
+F0 "PC" 60
+F1 "PC.sch" 60
+$EndSheet
+$Sheet
+S -4500 -4150 3950 2250
+U 5A2188BF
+F0 "Registers" 60
+F1 "Registers.sch" 60
+$EndSheet
 $EndSCHEMATC
