File: Computer/ALU.sch (KiCad schematic (older format))
At the start: 21 parts, among them J1 Conn_01x08, J2 Conn_01x08, J3 Conn_01x04, J4 Conn_01x01, J5 Conn_01x08, U1 74LS253, U10 74LS08, U11 74LS283, U12 74LS283, U13 74LS257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

Commit message: computer changes
Parts:
- removed J2, J5: Conn_01x08, Pin_Headers:Pin_Header_Angled_1x08_Pitch2.00mm, symbol Conn_01x08
- added J2, J5, J6: Conn_01x01, Pin_Headers:Pin_Header_Angled_1x01_Pitch1.00mm, symbol Conn_01x01
- added U17, U18: 74LS574, symbol 74LS574
Connections:
- net A0: now also U17.19 (Q0); no longer J1.8 (Pin_8)
- net A1: now also U17.18 (Q1); no longer J1.7 (Pin_7)
- net A2: now also U17.17 (Q2); no longer J1.6 (Pin_6)
- net A3: now also U17.16 (Q3); no longer J1.5 (Pin_5)
- net A4: now also U17.15 (Q4); no longer J1.4 (Pin_4)
- net A5: now also U17.14 (Q5); no longer J1.3 (Pin_3)
- net A6: now also U17.13 (Q6); no longer J1.2 (Pin_2)
- net A7: now also U17.12 (Q7); no longer J1.1 (Pin_1)
- net GND: now also U17.1 (OE), U17.10 (GND), U18.10 (GND)
- net OUT0: now also U18.2 (D0)
- net OUT1: now also U18.3 (D1)
- net OUT2: now also U18.4 (D2)
- net OUT3: now also U18.5 (D3)
- net OUT4: now also U18.6 (D4)
- net OUT5: now also U18.7 (D5)
- net OUT6: now also U18.8 (D6)
- net OUT7: now also U18.9 (D7)
- net VCC: now also U17.20 (VCC), U18.20 (VCC)
- net B0 renamed BUS0
- net BUS0: now also J1.8 (Pin_8), U17.2 (D0), U18.19 (Q0)
- net B1 renamed BUS1
- net BUS1: now also J1.7 (Pin_7), U17.3 (D1), U18.18 (Q1)
- net B2 renamed BUS2
- net BUS2: now also J1.6 (Pin_6), U17.4 (D2), U18.17 (Q2)
- net B3 renamed BUS3
- net BUS3: now also J1.5 (Pin_5), U17.5 (D3), U18.16 (Q3)
- net B4 renamed BUS4
- net BUS4: now also J1.4 (Pin_4), U17.6 (D4), U18.15 (Q4)
- net B5 renamed BUS5
- net BUS5: now also J1.3 (Pin_3), U17.7 (D5), U18.14 (Q5)
- net B6 renamed BUS6
- net BUS6: now also J1.2 (Pin_2), U17.8 (D6), U18.13 (Q6)
- net B7 renamed BUS7
- net BUS7: now also J1.1 (Pin_1), U17.9 (D7), U18.12 (Q7)
- new net AL: J2.1 (Pin_1), U17.11 (Cp)
- new net OB: J6.1 (Pin_1), U18.1 (OE)
- new net OL: J5.1 (Pin_1), U18.11 (Cp)
Other:
- moved on the sheet: J3, J4, U1, U10A, U10B, U11, U12, U13, U14, U15, U16, U2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

Commit message: updates
Parts:
- removed U15, U16: 74LS257, Housings_DIP:DIP-16_W7.62mm, symbol 74LS257
- removed unit 2 of U9
- added unit 3 of U10
- added unit 4 of U10
- added U15: 74LS04, Housings_DIP:DIP-14_W7.62mm, symbol 74LS04
- added U16: 74LS244, Housings_DIP:DIP-14_W7.62mm, symbol 74LS244
- J1: footprint Pin_Headers:Pin_Header_Angled_1x08_Pitch2.00mm -> Pin_Headers:Pin_Header_Straight_1x08_Pitch1.00mm
- J2: footprint Pin_Headers:Pin_Header_Angled_1x01_Pitch1.00mm -> Pin_Headers:Pin_Header_Straight_1x01_Pitch2.00mm
- J3: footprint Pin_Headers:Pin_Header_Angled_1x04_Pitch2.00mm -> Pin_Headers:Pin_Header_Straight_1x04_Pitch1.00mm
- J4, J5, J6: footprint Pin_Headers:Pin_Header_Angled_1x01_Pitch1.00mm -> Pin_Headers:Pin_Header_Straight_1x01_Pitch1.00mm
- U17, U18: footprint (none) -> Housings_DIP:DIP-14_W7.62mm
- U9: footprint Housings_DIP:DIP-14_W7.62mm -> Housings_DIP:DIP-16_W7.62mm
Connections:
- net GND: now also U10.7 (GND), U10.7 (GND), U15.7 (GND), U15.7 (GND), U15.7 (GND), U16.10 (GND); no longer U13.15 (OE), U14.15 (OE)
- net OUT0: now also U13.4 (Za), U16.18 (O0a)
- net OUT1: now also U13.7 (Zb), U16.16 (O1a)
- net OUT2: now also U13.12 (Zc), U16.14 (O2a)
- net OUT3: now also U13.9 (Zd), U16.12 (O3a)
- net OUT4: now also U14.4 (Za), U16.9 (O0b)
- net OUT5: now also U14.7 (Zb), U16.7 (O1b)
- net OUT6: now also U14.12 (Zc), U16.5 (O2b)
- net OUT7: now also U14.9 (Zd), U16.3 (O3b)
- net S2: now also U10.10, U15.5
- net S3: now also U10.12, U10.9
- net VCC: now also U10.14 (VCC), U10.14 (VCC), U15.14 (VCC), U15.14 (VCC), U15.14 (VCC), U16.20 (VCC)
- net at U11.1 (S2): now also U16.4 (I1a)
- net at U11.10 (S4): now also U16.8 (I3a)
- net at U11.13 (S3): now also U16.6 (I2a)
- net at U11.4 (S1): now also U16.2 (I0a)
- net at U12.1 (S2): now also U16.13 (I1b)
- net at U12.10 (S4): now also U16.17 (I3b)
- net at U12.13 (S3): now also U16.15 (I2b)
- net at U12.4 (S1): now also U16.11 (I0b)
- new net: U13.15 (OE), U14.15 (OE), U15.2
- new net: U15.4, U16.1 (OEa), U16.19 (OEb)
- new net: U10.8, U15.1
- new net: U10.13, U15.6
- new net: U10.11, U15.3
Other:
- moved on the sheet: J1, J2, J4, J5, J6, U10A, U10B, U11, U12, U13, U14, U17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
