File: Computer/Computer.kicad_pcb (KiCad board)
At the start: 2 copper layers, 21 parts, among them J1 Conn_01x08, J2 Conn_01x08, J3 Conn_01x04, J4 Conn_01x01, J5 Conn_01x08, U1 74LS253, U10 74LS08, U11 74LS283, U12 74LS283, U13 74LS257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

Commit message: updates
Parts:
- added J6: Conn_01x01, Pin_Headers:Pin_Header_Angled_1x01_Pitch1.00mm, F.Cu at (161.0, -7.82)
- added U17: 74LS574, Housings_DIP:DIP-14_W7.62mm, F.Cu at (-10.3, 105.8)
- added U18: 74LS574, Housings_DIP:DIP-14_W7.62mm, F.Cu at (177.9, -10.5)
- added U19: 74LS574, Housings_DIP:DIP-14_W7.62mm, F.Cu at (146.3, -14.0)
- added U20: 74LS161, Housings_DIP:DIP-14_W7.62mm, F.Cu at (217.1, 4.83)
- added U21: 74LS154, Housings_DIP:DIP-14_W7.62mm, F.Cu at (229.7, 3.58)
- added U22: 74LS154, Housings_DIP:DIP-14_W7.62mm, F.Cu at (169.3, -18.2)
- added U23, U24, U25, U26, U27, U28, U29, U30, U31, U32, U33, U34, U35, U36, U37, U38: 74LS574, Housings_DIP:DIP-14_W7.62mm, F.Cu at (161.0, -7.82)
- J2, J5: value Conn_01x08 -> Conn_01x01
- U15: value 74LS257 -> 74LS04
- U16: value 74LS257 -> 74LS244
- moved J1 114.2 mm to (-44.8, 123.4)
Connections:
- J1 pad 1: /ALU/A7 -> /ALU/BUS7
- J1 pad 2: /ALU/A6 -> /ALU/BUS6
- J1 pad 3: /ALU/A5 -> /ALU/BUS5
- J1 pad 4: /ALU/A4 -> /ALU/BUS4
- J1 pad 5: /ALU/A3 -> /ALU/BUS3
- J1 pad 6: /ALU/A2 -> /ALU/BUS2
- J1 pad 7: /ALU/A1 -> /ALU/BUS1
- J1 pad 8: /ALU/A0 -> /ALU/BUS0
- J2 pad 1: /ALU/B7 -> /ALU/AL
- J2 pad 2: /ALU/B6 -> (no net)
- J2 pad 3: /ALU/B5 -> (no net)
- J2 pad 4: /ALU/B4 -> (no net)
- J2 pad 5: /ALU/B3 -> (no net)
- J2 pad 6: /ALU/B2 -> (no net)
- J2 pad 7: /ALU/B1 -> (no net)
- J2 pad 8: /ALU/B0 -> (no net)
- J5 pad 1: /ALU/OUT0 -> /ALU/OL
- J5 pad 2: /ALU/OUT1 -> (no net)
- J5 pad 3: /ALU/OUT2 -> (no net)
- J5 pad 4: /ALU/OUT3 -> (no net)
- J5 pad 5: /ALU/OUT4 -> (no net)
- J5 pad 6: /ALU/OUT5 -> (no net)
- J5 pad 7: /ALU/OUT6 -> (no net)
- J5 pad 8: /ALU/OUT7 -> (no net)
- U1 pad 2: /ALU/B0 -> /ALU/BUS0
- U10 pad 10: (no net) -> /ALU/S2
- U10 pad 11: (no net) -> Net-(U10-Pad11)
- U10 pad 12: (no net) -> /ALU/S3
- U10 pad 13: (no net) -> Net-(U10-Pad13)
- U10 pad 8: (no net) -> Net-(U10-Pad8)
- U10 pad 9: (no net) -> /ALU/S3
- U13 pad 12: Net-(U13-Pad12) -> /ALU/OUT2
- U13 pad 15: GND -> Net-(U13-Pad15)
- U13 pad 4: Net-(U13-Pad4) -> /ALU/OUT0
- U13 pad 7: Net-(U13-Pad7) -> /ALU/OUT1
- U13 pad 9: Net-(U13-Pad9) -> /ALU/OUT3
- U14 pad 12: Net-(U14-Pad12) -> /ALU/OUT6
- U14 pad 15: GND -> Net-(U13-Pad15)
- U14 pad 4: Net-(U14-Pad4) -> /ALU/OUT4
- U14 pad 7: Net-(U14-Pad7) -> /ALU/OUT5
- U14 pad 9: Net-(U14-Pad9) -> /ALU/OUT7
- U15 pad 1: /ALU/S2 -> Net-(U10-Pad8)
- U15 pad 10: Net-(U13-Pad9) -> (no net)
- U15 pad 11: Net-(U11-Pad10) -> (no net)
- U15 pad 12: /ALU/OUT2 -> (no net)
- U15 pad 13: Net-(U13-Pad12) -> (no net)
- U15 pad 14: Net-(U11-Pad13) -> VCC
- U15 pad 15: Net-(U15-Pad15) -> (no net)
- U15 pad 16: VCC -> (no net)
- U15 pad 2: Net-(U11-Pad4) -> Net-(U13-Pad15)
- U15 pad 3: Net-(U13-Pad4) -> Net-(U10-Pad11)
- U15 pad 4: /ALU/OUT0 -> Net-(U15-Pad4)
- U15 pad 5: Net-(U11-Pad1) -> /ALU/S2
- U15 pad 6: Net-(U13-Pad7) -> Net-(U10-Pad13)
- U15 pad 7: /ALU/OUT1 -> GND
- U15 pad 8: GND -> (no net)
- U15 pad 9: /ALU/OUT3 -> (no net)
- U16 pad 1: /ALU/S2 -> Net-(U15-Pad4)
- U16 pad 10: Net-(U14-Pad9) -> GND
- U16 pad 11: Net-(U12-Pad10) -> Net-(U12-Pad4)
- U16 pad 12: /ALU/OUT6 -> /ALU/OUT3
- U16 pad 13: Net-(U14-Pad12) -> Net-(U12-Pad1)
- U16 pad 14: Net-(U12-Pad13) -> /ALU/OUT2
- U16 pad 15: Net-(U15-Pad15) -> Net-(U12-Pad13)
- U16 pad 16: VCC -> /ALU/OUT1
- U16 pad 2: Net-(U12-Pad4) -> Net-(U11-Pad4)
- U16 pad 3: Net-(U14-Pad4) -> /ALU/OUT7
- U16 pad 4: /ALU/OUT4 -> Net-(U11-Pad1)
- U16 pad 5: Net-(U12-Pad1) -> /ALU/OUT6
- U16 pad 6: Net-(U14-Pad7) -> Net-(U11-Pad13)
- U16 pad 8: GND -> Net-(U11-Pad10)
- U16 pad 9: /ALU/OUT7 -> /ALU/OUT4
- U2 pad 2: /ALU/B1 -> /ALU/BUS1
- U3 pad 2: /ALU/B2 -> /ALU/BUS2
- U4 pad 2: /ALU/B3 -> /ALU/BUS3
- U5 pad 2: /ALU/B4 -> /ALU/BUS4
- U6 pad 2: /ALU/B5 -> /ALU/BUS5
- U7 pad 2: /ALU/B6 -> /ALU/BUS6
- U8 pad 2: /ALU/B7 -> /ALU/BUS7
- U9 pad 3: /ALU/S3 -> (no net)
- U9 pad 4: Net-(U15-Pad15) -> (no net)
Routing:
- net /ALU/S2: track 0.00 -> 164.2 mm
- net /ALU/S3: track 0.00 -> 102.9 mm, vias 0 -> 5
- net /ALU/S1: track 0.00 -> 71.9 mm, vias 0 -> 2
- net /ALU/S0: track 0.00 -> 41.8 mm, vias 0 -> 2
