File: Computer/PC.sch (KiCad schematic (older format))
At the start: 2 parts

Commit message: updates
Parts:
- U19, U20: renamed from U?; footprint (none) -> Housings_DIP:DIP-14_W7.62mm
Changed lines of the file:
@@
 $EndDescr
 $Comp
-L 74LS574 U?
+L 74LS574 U19
 U 1 1 5A21883F
 P 1700 3300
-F 0 "U?" H 1700 3300 50  0000 C CNN
+F 0 "U19" H 1700 3300 50  0000 C CNN
 F 1 "74LS574" H 1750 2950 50  0000 C CNN
-F 2 "" H 1700 3300 50  0001 C CNN
+F 2 "Housings_DIP:DIP-14_W7.62mm" H 1700 3300 50  0001 C CNN
 F 3 "" H 1700 3300 50  0001 C CNN
 	1    1700 3300
@@
 $EndComp
 $Comp
-L 74LS161 U?
+L 74LS161 U20
 U 1 1 5A218866
 P 3200 4950
-F 0 "U?" H 3250 5050 50  0000 C CNN
+F 0 "U20" H 3250 5050 50  0000 C CNN
 F 1 "74LS161" H 3300 4750 50  0000 C CNN
-F 2 "" H 3200 4950 50  0001 C CNN
+F 2 "Housings_DIP:DIP-14_W7.62mm" H 3200 4950 50  0001 C CNN
 F 3 "" H 3200 4950 50  0001 C CNN
 	1    3200 4950
