File: Computer/Registers.sch (KiCad schematic (older format))
At the start: 4 parts

Commit message: update
Parts:
- added U? (x12): 74LS574, symbol 74LS574
- added U?: 74LS154, symbol 74LS154
Connections:
- net GND: now also U?.10 (GND), U?.10 (GND), U?.10 (GND), U?.10 (GND), U?.10 (GND), U?.10 (GND), U?.10 (GND), U?.10 (GND), U?.10 (GND), U?.10 (GND), U?.10 (GND), U?.10 (GND), U?.12 (GND)
- net VCC: now also U?.20 (VCC), U?.20 (VCC), U?.20 (VCC), U?.20 (VCC), U?.20 (VCC), U?.20 (VCC), U?.20 (VCC), U?.20 (VCC), U?.20 (VCC), U?.20 (VCC), U?.20 (VCC), U?.20 (VCC), U?.24 (VCC)
Other:
- moved on the sheet: U?
Changed lines of the file:
@@
 L 74LS574 U?
 U 1 1 5A2188CC
-P 2150 2700
-F 0 "U?" H 2150 2700 50  0000 C CNN
-F 1 "74LS574" H 2200 2350 50  0000 C CNN
-F 2 "" H 2150 2700 50  0001 C CNN
-F 3 "" H 2150 2700 50  0001 C CNN
-	1    2150 2700
+P 4800 1300
+F 0 "U?" H 4800 1300 50  0000 C CNN
+F 1 "74LS574" H 4850 950 50  0000 C CNN
+F 2 "" H 4800 1300 50  0001 C CNN
+F 3 "" H 4800 1300 50  0001 C CNN
+	1    4800 1300
 	1    0    0    -1
 $EndComp
@@
 L 74LS574 U?
 U 1 1 5A21893B
-P 2150 4000
-F 0 "U?" H 2150 4000 50  0000 C CNN
-F 1 "74LS574" H 2200 3650 50  0000 C CNN
-F 2 "" H 2150 4000 50  0001 C CNN
-F 3 "" H 2150 4000 50  0001 C CNN
-	1    2150 4000
+P 4800 2600
+F 0 "U?" H 4800 2600 50  0000 C CNN
+F 1 "74LS574" H 4850 2250 50  0000 C CNN
+F 2 "" H 4800 2600 50  0001 C CNN
+F 3 "" H 4800 2600 50  0001 C CNN
+	1    4800 2600
 	1    0    0    -1
 $EndComp
@@
 L 74LS574 U?
 U 1 1 5A2189B0
-P 2150 5300
-F 0 "U?" H 2150 5300 50  0000 C CNN
-F 1 "74LS574" H 2200 4950 50  0000 C CNN
-F 2 "" H 2150 5300 50  0001 C CNN
-F 3 "" H 2150 5300 50  0001 C CNN
-	1    2150 5300
+P 4800 3900
+F 0 "U?" H 4800 3900 50  0000 C CNN
+F 1 "74LS574" H 4850 3550 50  0000 C CNN
+F 2 "" H 4800 3900 50  0001 C CNN
+F 3 "" H 4800 3900 50  0001 C CNN
+	1    4800 3900
 	1    0    0    -1
 $EndComp
@@
 L 74LS574 U?
 U 1 1 5A218A0D
-P 2150 6600
-F 0 "U?" H 2150 6600 50  0000 C CNN
-F 1 "74LS574" H 2200 6250 50  0000 C CNN
-F 2 "" H 2150 6600 50  0001 C CNN
-F 3 "" H 2150 6600 50  0001 C CNN
-	1    2150 6600
+P 4800 5200
+F 0 "U?" H 4800 5200 50  0000 C CNN
+F 1 "74LS574" H 4850 4850 50  0000 C CNN
+F 2 "" H 4800 5200 50  0001 C CNN
+F 3 "" H 4800 5200 50  0001 C CNN
+	1    4800 5200
 	1    0    0    -1
 $EndComp
+$Comp
+L 74LS574 U?
+U 1 1 5A2228E2
+P 6650 1300
+F 0 "U?" H 6650 1300 50  0000 C CNN
+F 1 "74LS574" H 6700 950 50  0000 C CNN
+F 2 "" H 6650 1300 50  0001 C CNN
+F 3 "" H 6650 1300 50  0001 C CNN
+	1    6650 1300
+	1    0    0    -1
+$EndComp
+$Comp
+L 74LS574 U?
+U 1 1 5A2228E8
+P 6650 2600
+F 0 "U?" H 6650 2600 50  0000 C CNN
+F 1 "74LS574" H 6700 2250 50  0000 C CNN
+F 2 "" H 6650 2600 50  0001 C CNN
+F 3 "" H 6650 2600 50  0001 C CNN
+	1    6650 2600
+	1    0    0    -1
+$EndComp
+$Comp
+L 74LS574 U?
+U 1 1 5A2228EE
+P 6650 3900
+F 0 "U?" H 6650 3900 50  0000 C CNN
+F 1 "74LS574" H 6700 3550 50  0000 C CNN
+F 2 "" H 6650 3900 50  0001 C CNN
+F 3 "" H 6650 3900 50  0001 C CNN
+	1    6650 3900
+	1    0    0    -1
+$EndComp
+$Comp
+L 74LS574 U?
+U 1 1 5A2228F4
+P 6650 5200
+F 0 "U?" H 6650 5200 50  0000 C CNN
+F 1 "74LS574" H 6700 4850 50  0000 C CNN
+F 2 "" H 6650 5200 50  0001 C CNN
+F 3 "" H 6650 5200 50  0001 C CNN
+	1    6650 5200
+	1    0    0    -1
+$EndComp
+$Comp
+L 74LS574 U?
+U 1 1 5A222A06
+P 8450 1300
+F 0 "U?" H 8450 1300 50  0000 C CNN
+F 1 "74LS574" H 8500 950 50  0000 C CNN
+F 2 "" H 8450 1300 50  0001 C CNN
+F 3 "" H 8450 1300 50  0001 C CNN
+	1    8450 1300
+	1    0    0    -1
+$EndComp
+$Comp
+L 74LS574 U?
+U 1 1 5A222A0C
+P 8450 2600
+F 0 "U?" H 8450 2600 50  0000 C CNN
+F 1 "74LS574" H 8500 2250 50  0000 C CNN
+F 2 "" H 8450 2600 50  0001 C CNN
+F 3 "" H 8450 2600 50  0001 C CNN
+	1    8450 2600
+	1    0    0    -1
+$EndComp
+$Comp
+L 74LS574 U?
+U 1 1 5A222A12
+P 8450 3900
+F 0 "U?" H 8450 3900 50  0000 C CNN
+F 1 "74LS574" H 8500 3550 50  0000 C CNN
+F 2 "" H 8450 3900 50  0001 C CNN
+F 3 "" H 8450 3900 50  0001 C CNN
+	1    8450 3900
+	1    0    0    -1
+$EndComp
+$Comp
+L 74LS574 U?
+U 1 1 5A222A18
+P 8450 5200
+F 0 "U?" H 8450 5200 50  0000 C CNN
+F 1 "74LS574" H 8500 4850 50  0000 C CNN
+F 2 "" H 8450 5200 50  0001 C CNN
+F 3 "" H 8450 5200 50  0001 C CNN
+	1    8450 5200
+	1    0    0    -1
+$EndComp
+$Comp
+L 74LS574 U?
+U 1 1 5A222B3A
+P 10200 1300
+F 0 "U?" H 10200 1300 50  0000 C CNN
+F 1 "74LS574" H 10250 950 50  0000 C CNN
+F 2 "" H 10200 1300 50  0001 C CNN
+F 3 "" H 10200 1300 50  0001 C CNN
+	1    10200 1300
+	1    0    0    -1
+$EndComp
+$Comp
+L 74LS574 U?
+U 1 1 5A222B40
+P 10200 2600
+F 0 "U?" H 10200 2600 50  0000 C CNN
+F 1 "74LS574" H 10250 2250 50  0000 C CNN
+F 2 "" H 10200 2600 50  0001 C CNN
+F 3 "" H 10200 2600 50  0001 C CNN
+	1    10200 2600
+	1    0    0    -1
+$EndComp
+$Comp
+L 74LS574 U?
+U 1 1 5A222B46
+P 10200 3900
+F 0 "U?" H 10200 3900 50  0000 C CNN
+F 1 "74LS574" H 10250 3550 50  0000 C CNN
+F 2 "" H 10200 3900 50  0001 C CNN
+F 3 "" H 10200 3900 50  0001 C CNN
+	1    10200 3900
+	1    0    0    -1
+$EndComp
+$Comp
+L 74LS574 U?
+U 1 1 5A222B4C
+P 10200 5200
+F 0 "U?" H 10200 5200 50  0000 C CNN
+F 1 "74LS574" H 10250 4850 50  0000 C CNN
+F 2 "" H 10200 5200 50  0001 C CNN
+F 3 "" H 10200 5200 50  0001 C CNN
+	1    10200 5200
+	1    0    0    -1
+$EndComp
+$Comp
+L 74LS154 U?
+U 1 1 5A222BE4
+P 2650 1500
+F 0 "U?" H 2650 2400 50  0000 C CNN
+F 1 "74LS154" H 2600 650 50  0000 C CNN
+F 2 "" H 2650 1500 50  0001 C CNN
+F 3 "" H 2650 1500 50  0001 C CNN
+	1    2650 1500
+	1    0    0    -1
+$EndComp

Commit message: updates
Parts:
- added U22: 74LS154, Housings_DIP:DIP-14_W7.62mm, symbol 74LS154
- U21, U23, U24, U25, U26, U27, U28, U29, U30, U31, U32, U33, U34, U35, U36, U37, U38: renamed from U?; footprint (none) -> Housings_DIP:DIP-14_W7.62mm
Connections:
- net GND: now also U22.12 (GND)
- net VCC: now also U22.24 (VCC)
Other:
- moved on the sheet: U21, U23, U24, U25, U26, U27, U28, U29, U30, U31, U32, U33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
