File: 4 bit alu/4 bit alu.sch (KiCad schematic (older format))
At the start: 19 parts, among them J1 Conn_01x01, J2 Conn_01x04, J4 Conn_01x01, SW1 SW_Coded, SW2 SW_Coded, SW3 SW_Coded, U1 74LS253, U10 74LS08, U11 74LS283, U13 74LS257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

Commit message: update
Connections:
- net S0: no longer U10.6
- net A4: no longer names the net of U13.11 (I0d)
- net A4: now also U10.6
- no-connect marks 0 -> 1
Changed lines of the file:
@@
 LIBS:contrib
 LIBS:valves
+LIBS:4 bit alu-cache
 EELAYER 25 0
 EELAYER END
@@
 	5500 3650 5600 3750
 Entry Wire Line
-	5500 3800 5600 3900
-Entry Wire Line
 	5500 3900 5600 4000
 Text Label 5700 4150 0    60   ~ 0
@@
 Text Label 5650 3750 0    60   ~ 0
 A1
-Text Label 5650 3900 0    60   ~ 0
-A4
 Text Label 5650 4000 0    60   ~ 0
 A2
@@
 	5600 4000 5700 4000
 Wire Wire Line
-	5700 3900 5600 3900
-Wire Wire Line
 	5600 3750 5700 3750
 Wire Wire Line
@@
 $EndComp
 Wire Wire Line
-	5700 4150 5400 4150
-Wire Wire Line
-	5400 4150 5400 4400
+	5400 3850 5400 4400
 Wire Wire Line
 	5400 4400 6950 4400
+NoConn ~ 7100 2150
+Wire Wire Line
+	5400 3850 5700 3850
+Wire Wire Line
+	5700 3850 5700 3900
 $EndSCHEMATC
