File: ledTree/ledTree.sch (KiCad schematic (older format))
At the start: 14 parts, among them SW1 SW_Push, U1 ATTINY85, U10 WS2812b, U11 WS2812b, U12 WS2812b, U13 WS2812b, U2 WS2812b, U3 WS2812b, U4 WS2812b, U5 WS2812b, U6 WS2812b, U7 WS2812b, U8 WS2812b, U9 WS2812b

Commit message: finished tree!
Parts:
- added J1: OUT1, Connectors:Pin_d0.9mm_L10.0mm_W2.4mm_FlatFork, symbol Conn_01x01
- added J10, J9: VCC, Connectors:Pin_d0.9mm_L10.0mm_W2.4mm_FlatFork, symbol Conn_01x01
- added J2: IN1, Connectors:Pin_d0.9mm_L10.0mm_W2.4mm_FlatFork, symbol Conn_01x01
- added J3: OUT2, Connectors:Pin_d0.9mm_L10.0mm_W2.4mm_FlatFork, symbol Conn_01x01
- added J4: IN2, Connectors:Pin_d0.9mm_L10.0mm_W2.4mm_FlatFork, symbol Conn_01x01
- added J5: OUT3, Connectors:Pin_d0.9mm_L10.0mm_W2.4mm_FlatFork, symbol Conn_01x01
- added J6: IN3, Connectors:Pin_d0.9mm_L10.0mm_W2.4mm_FlatFork, symbol Conn_01x01
- added J7, J8: GND, Connectors:Pin_d0.9mm_L10.0mm_W2.4mm_FlatFork, symbol Conn_01x01
- added U13, U17, U5, U9: WS2812b, LEDs:LED_D5.0mm-4, symbol WS2812b
- U1: footprint (none) -> ledTree:ATTINY85
- renumbered U4 to U10, U8 to U11, U5 to U14, U9 to U15, U13 to U16, U6 to U3, U10 to U4, U3 to U6, U11 to U8
Connections:
- net GND: now also J7.1 (Pin_1), J8.1 (Pin_1), U13.2 (GND), U17.2 (GND), U5.2 (GND), U9.2 (GND)
- net VCC: now also J10.1 (Pin_1), J9.1 (Pin_1), U13.3 (Vcc), U17.3 (Vcc), U5.3 (Vcc), U9.3 (Vcc)
- net at U4.1 (Dout): now also U5.4 (Din); no longer U6.4 (Din)
- net at U8.1 (Dout): now also U9.4 (Din); no longer U10.4 (Din)
- net at U12.1 (Dout): now also U13.4 (Din); no longer U14.4 (Din)
- net at U16.1 (Dout): now also U17.4 (Din)
- new net IN1: J2.1 (Pin_1), U6.4 (Din)
- new net IN2: J4.1 (Pin_1), U10.4 (Din)
- new net IN3: J6.1 (Pin_1), U14.4 (Din)
- new net OUT1: J1.1 (Pin_1), U5.1 (Dout)
- new net OUT2: J3.1 (Pin_1), U9.1 (Dout)
- new net OUT3: J5.1 (Pin_1), U13.1 (Dout)
Other:
- moved on the sheet: SW1, U1
