File: ledTree/ledTree.sch (KiCad schematic (older format))
At the start: 29 parts, among them J1 OUT1, J10 VCC, J2 IN1, J3 OUT2, J4 IN2, J5 OUT3, J6 IN3, J7 GND, J8 GND, J9 VCC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

Commit message: update
Parts:
- added C1: CP, Capacitors_THT:CP_Radial_D5.0mm_P2.50mm, symbol CP
- RV1: renamed from RV?; footprint (none) -> Potentiometers:Potentiometer_Trimmer_Bourns_3339S_Vertical
Connections:
- net GND: now also C1.2
- net VCC: now also C1.1
Changed lines of the file:
@@
 VCC
 $Comp
-L POT RV?
+L POT RV1
 U 1 1 5A2479DB
 P 3450 1900
-F 0 "RV?" V 3275 1900 50  0000 C CNN
+F 0 "RV1" V 3275 1900 50  0000 C CNN
 F 1 "POT" V 3350 1900 50  0000 C CNN
-F 2 "" H 3450 1900 50  0001 C CNN
+F 2 "Potentiometers:Potentiometer_Trimmer_Bourns_3339S_Vertical" H 3450 1900 50  0001 C CNN
 F 3 "" H 3450 1900 50  0001 C CNN
 	1    3450 1900
@@
 Wire Wire Line
 	3700 2500 4200 2500
+$Comp
+L CP C1
+U 1 1 5A2482EF
+P 4200 1400
+F 0 "C1" H 4225 1500 50  0000 L CNN
+F 1 "CP" H 4225 1300 50  0000 L CNN
+F 2 "Capacitors_THT:CP_Radial_D5.0mm_P2.50mm" H 4238 1250 50  0001 C CNN
+F 3 "" H 4200 1400 50  0001 C CNN
+	1    4200 1400
+	1    0    0    -1
+$EndComp
+Text GLabel 4200 1250 1    60   Input ~ 0
+VCC
+Text GLabel 4200 1550 3    60   Input ~ 0
+GND
 $EndSCHEMATC

Commit message: updates
Connections:
- net at U1.1 (PB1): now also SW1.2
- net at U1.5 (PB5): no longer SW1.2
- no-connect marks 5 -> 4
Changed lines of the file:
@@
 Text GLabel 2250 1800 0    60   Input ~ 0
 GND
-NoConn ~ 3250 1800
 $Comp
 L SW_Push SW1
@@
 	1    0    0    -1
 $EndComp
-Wire Wire Line
-	3250 2200 3300 2200
-Wire Wire Line
-	3300 2200 3300 2650
 Wire Wire Line
 	3300 2650 3150 2650
@@
 Text GLabel 4200 1550 3    60   Input ~ 0
 GND
+Wire Wire Line
+	3300 2650 3300 2300
+Wire Wire Line
+	3300 2300 2900 2300
+Wire Wire Line
+	2900 2300 2900 1800
+Wire Wire Line
+	2900 1800 3250 1800
 $EndSCHEMATC
