File: ledTree/_saved_ledTree.sch (KiCad schematic (older format))
At the start: 29 parts, among them J1 OUT1, J10 VCC, J2 IN1, J3 OUT2, J4 IN2, J5 OUT3, J6 IN3, J7 GND, J8 GND, J9 VCC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

Commit message: update
Parts:
- RV1: renamed from RV?; footprint (none) -> Potentiometers:Potentiometer_Trimmer_Bourns_3339S_Vertical
Changed lines of the file:
@@
 VCC
 $Comp
-L POT RV?
+L POT RV1
 U 1 1 5A2479DB
 P 3450 1900
-F 0 "RV?" V 3275 1900 50  0000 C CNN
+F 0 "RV1" V 3275 1900 50  0000 C CNN
 F 1 "POT" V 3350 1900 50  0000 C CNN
-F 2 "" H 3450 1900 50  0001 C CNN
+F 2 "Potentiometers:Potentiometer_Trimmer_Bourns_3339S_Vertical" H 3450 1900 50  0001 C CNN
 F 3 "" H 3450 1900 50  0001 C CNN
 	1    3450 1900
