File: ledTree/ledTree.kicad_pcb (KiCad board)
At the start: 2 copper layers, 124.5 x 115.6 mm, 13 parts, among them SW1 SW_Push, U10 WS2812b, U11 WS2812b, U12 WS2812b, U13 WS2812b, U2 WS2812b, U3 WS2812b, U4 WS2812b, U5 WS2812b, U6 WS2812b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

Commit message: update
Parts:
- moved U4 194.0 mm to (-72.6, 37.1)
- moved U8 159.7 mm to (-54.1, 103.4), turned to 90 degrees
- moved U2 156.2 mm to (-57.9, 82.0)
- moved U11 153.5 mm to (-67.1, 59.4)
Other:
- board size 124.5 x 115.6 mm -> 124.5 x 115.1 mm
Changed lines of the file:
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@@
     (links 36)
     (no_connects 36)
-    (area -86.435001 -0.075001 38.175001 115.645001)
+    (area -86.435001 -0.075001 38.175001 115.137001)
     (thickness 1.6)
-    (drawings 39)
+    (drawings 47)
     (tracks 0)
     (zones 0)
@@
     (pad_to_mask_clearance 0.2)
     (aux_axis_origin 0 0)
-    (visible_elements FFFFFF7F)
+    (visible_elements 7FFFFFFF)
     (pcbplotparams
       (layerselection 0x00030_80000001)
@@
   )
   (module LEDs:LED_D5.0mm-4 (layer F.Cu)
-    (at 96.52 105.41 90)
+    (at -57.912 82.042 90)
     (descr "LED, diameter 5.0mm, 2 pins, diameter 5.0mm, 3 pins, diameter 5.0mm, 4 pins, http://www.kingbright.com/attachments/file/psearch/000/00/00/L-154A4SUREQBFZGEW(Ver.9A).pdf")
     (tags "LED diameter 5.0mm 2 pins diameter 5.0mm 3 pins diameter 5.0mm 4 pins")
@@
   )
   (module LEDs:LED_D5.0mm-4 (layer F.Cu)
-    (at 96.52 132.08)
+    (at -72.644 37.084)
     (descr "LED, diameter 5.0mm, 2 pins, diameter 5.0mm, 3 pins, diameter 5.0mm, 4 pins, http://www.kingbright.com/attachments/file/psearch/000/00/00/L-154A4SUREQBFZGEW(Ver.9A).pdf")
     (tags "LED diameter 5.0mm 2 pins diameter 5.0mm 3 pins diameter 5.0mm 4 pins")
@@
   )
   (module LEDs:LED_D5.0mm-4 (layer F.Cu)
-    (at 105.419762 95.995)
-    (descr "LED, diameter 5.0mm, 2 pins, diameter 5.0mm, 3 pins, diameter 5.0mm, 4 pins, http://www.kingbright.com/attachments/file/psearch/000/00/00/L-154A4SUREQBFZGEW(Ver.9A).pdf")
-    (tags "LED diameter 5.0mm 2 pins diameter 5.0mm 3 pins diameter 5.0mm 4 pins")
-    (fp_text reference U8 (at 1.905 -3.96) (layer F.SilkS)
-      (effects (font (size 1 1) (thickness 0.15)))
-    )
-    (fp_text value WS2812b (at 1.905 3.96) (layer F.Fab)
-      (effects (font (size 1 1) (thickness 0.15)))
-    )
-    (fp_arc (start 1.905 0) (end -0.595 -1.469694) (angle 299.1) (layer F.Fab) (width 0.1))
-    (fp_arc (start 1.905 0) (end -0.655 -1.54483) (angle 127.7) (layer F.SilkS) (width 0.12))
-    (fp_arc (start 1.905 0) (end -0.655 1.54483) (angle -127.7) (layer F.SilkS) (width 0.12))
-    (fp_arc (start 1.905 0) (end -0.349684 -1.08) (angle 128.8) (layer F.SilkS) (width 0.12))
-    (fp_arc (start 1.905 0) (end -0.349684 1.08) (angle -128.8) (layer F.SilkS) (width 0.12))
-    (fp_circle (center 1.905 0) (end 4.405 0) (layer F.Fab) (width 0.1))
-    (fp_line (start -0.595 -1.469694) (end -0.595 1.469694) (layer F.Fab) (width 0.1))
-    (fp_line (start -0.655 -1.545) (end -0.655 -1.08) (layer F.SilkS) (width 0.12))
-    (fp_line (start -0.655 1.08) (end -0.655 1.545) (layer F.SilkS) (width 0.12))
-    (fp_line (start -1.35 -3.25) (end -1.35 3.25) (layer F.CrtYd) (width 0.05))
-    (fp_line (start -1.35 3.25) (end 5.15 3.25) (layer F.CrtYd) (width 0.05))
-    (fp_line (start 5.15 3.25) (end 5.15 -3.25) (layer F.CrtYd) (width 0.05))
-    (fp_line (start 5.15 -3.25) (end -1.35 -3.25) (layer F.CrtYd) (width 0.05))
-    (pad 1 thru_hole rect (at 0 0) (size 1.07 1.8) (drill 0.9) (layers *.Cu *.Mask)
+    (at -54.102 103.378 90)
+    (descr "LED, diameter 5.0mm, 2 pins, diameter 5.0mm, 3 pins, diameter 5.0mm, 4 pins, http://www.kingbright.com/attachments/file/psearch/000/00/00/L-154A4SUREQBFZGEW(Ver.9A).pdf")
+    (tags "LED diameter 5.0mm 2 pins diameter 5.0mm 3 pins diameter 5.0mm 4 pins")
+    (fp_text reference U8 (at 1.905 -3.96 90) (layer F.SilkS)
+      (effects (font (size 1 1) (thickness 0.15)))
+    )
+    (fp_text value WS2812b (at 1.905 3.96 90) (layer F.Fab)
+      (effects (font (size 1 1) (thickness 0.15)))
+    )
+    (fp_arc (start 1.905 0) (end -0.595 -1.469694) (angle 299.1) (layer F.Fab) (width 0.1))
+    (fp_arc (start 1.905 0) (end -0.655 -1.54483) (angle 127.7) (layer F.SilkS) (width 0.12))
+    (fp_arc (start 1.905 0) (end -0.655 1.54483) (angle -127.7) (layer F.SilkS) (width 0.12))
+    (fp_arc (start 1.905 0) (end -0.349684 -1.08) (angle 128.8) (layer F.SilkS) (width 0.12))
+    (fp_arc (start 1.905 0) (end -0.349684 1.08) (angle -128.8) (layer F.SilkS) (width 0.12))
+    (fp_circle (center 1.905 0) (end 4.405 0) (layer F.Fab) (width 0.1))
+    (fp_line (start -0.595 -1.469694) (end -0.595 1.469694) (layer F.Fab) (width 0.1))
+    (fp_line (start -0.655 -1.545) (end -0.655 -1.08) (layer F.SilkS) (width 0.12))
+    (fp_line (start -0.655 1.08) (end -0.655 1.545) (layer F.SilkS) (width 0.12))
+    (fp_line (start -1.35 -3.25) (end -1.35 3.25) (layer F.CrtYd) (width 0.05))
+    (fp_line (start -1.35 3.25) (end 5.15 3.25) (layer F.CrtYd) (width 0.05))
+    (fp_line (start 5.15 3.25) (end 5.15 -3.25) (layer F.CrtYd) (width 0.05))
+    (fp_line (start 5.15 -3.25) (end -1.35 -3.25) (layer F.CrtYd) (width 0.05))
+    (pad 1 thru_hole rect (at 0 0 90) (size 1.07 1.8) (drill 0.9) (layers *.Cu *.Mask)
       (net 9 "Net-(U4-Pad4)"))
-    (pad 2 thru_hole oval (at 1.27 0) (size 1.07 1.8) (drill 0.9) (layers *.Cu *.Mask)
-      (net 4 VCC))
-    (pad 3 thru_hole oval (at 2.54 0) (size 1.07 1.8) (drill 0.9) (layers *.Cu *.Mask)
-      (net 2 GND))
-    (pad 4 thru_hole oval (at 3.81 0) (size 1.07 1.8) (drill 0.9) (layers *.Cu *.Mask)
+    (pad 2 thru_hole oval (at 1.27 0 90) (size 1.07 1.8) (drill 0.9) (layers *.Cu *.Mask)
+      (net 4 VCC))
+    (pad 3 thru_hole oval (at 2.54 0 90) (size 1.07 1.8) (drill 0.9) (layers *.Cu *.Mask)
+      (net 2 GND))
+    (pad 4 thru_hole oval (at 3.81 0 90) (size 1.07 1.8) (drill 0.9) (layers *.Cu *.Mask)
       (net 14 "Net-(U12-Pad1)"))
     (model ${KISYS3DMOD}/LEDs.3dshapes/LED_D5.0mm-4.wrl
@@
   )
   (module LEDs:LED_D5.0mm-4 (layer F.Cu)
-    (at 82.55 93.98)
+    (at -67.056 59.436)
     (descr "LED, diameter 5.0mm, 2 pins, diameter 5.0mm, 3 pins, diameter 5.0mm, 4 pins, http://www.kingbright.com/attachments/file/psearch/000/00/00/L-154A4SUREQBFZGEW(Ver.9A).pdf")
     (tags "LED diameter 5.0mm 2 pins diameter 5.0mm 3 pins diameter 5.0mm 4 pins")
@@
     )
   )
-  (gr_line (start -46.99 62.23) (end -49.53 62.23) (angle 90) (layer Edge.Cuts) (width 0.15))
+  (gr_line (start -55.88 104.14) (end -48.514 115.062) (angle 90) (layer Edge.Cuts) (width 0.15))
+  (gr_line (start -63.5 92.71) (end -59.436 98.806) (angle 90) (layer Edge.Cuts) (width 0.15))
+  (gr_line (start -55.118 104.14) (end -55.88 104.14) (angle 90) (layer Edge.Cuts) (width 0.15))
+  (gr_line (start -55.118 98.806) (end -55.118 104.14) (angle 90) (layer Edge.Cuts) (width 0.15))
+  (gr_line (start -59.436 98.806) (end -55.118 98.806) (angle 90) (layer Edge.Cuts) (width 0.15))
+  (gr_line (start -48.514 24.13) (end -48.006 24.13) (angle 90) (layer Edge.Cuts) (width 0.15))
+  (gr_line (start -48.514 59.69) (end -48.006 59.69) (angle 90) (layer Edge.Cuts) (width 0.15))
+  (gr_line (start -48.514 115.062) (end -48.514 59.69) (angle 90) (layer Edge.Cuts) (width 0.15))
+  (gr_line (start -48.006 67.31) (end -48.006 59.69) (angle 90) (layer Edge.Cuts) (width 0.15))
+  (gr_line (start -48.006 115.062) (end -48.006 67.31) (angle 90) (layer Edge.Cuts) (width 0.15))
+  (gr_line (start -48.006 115.062) (end -33.02 92.71) (angle 90) (layer Edge.Cuts) (width 0.15))
+  (gr_line (start -46.99 24.13) (end -48.006 24.13) (angle 90) (layer Edge.Cuts) (width 0.15))
+  (gr_line (start -48.514 24.13) (end -49.53 24.13) (angle 90) (layer Edge.Cuts) (width 0.15))
   (gr_line (start -46.99 24.13) (end -17.78 24.13) (angle 90) (layer Edge.Cuts) (width 0.15))
-  (gr_line (start -46.99 114.3) (end -46.99 24.13) (angle 90) (layer Edge.Cuts) (width 0.15))
-  (gr_line (start -49.53 24.13) (end -49.53 114.3) (angle 90) (layer Edge.Cuts) (width 0.15))
   (gr_line (start -50.8 24.13) (end -49.53 24.13) (angle 90) (layer Edge.Cuts) (width 0.15))
   (gr_line (start -78.74 24.13) (end -50.8 24.13) (angle 90) (layer Edge.Cuts) (width 0.15))
-  (gr_line (start -48.26 115.57) (end -33.02 92.71) (angle 90) (layer Edge.Cuts) (width 0.15))
   (gr_line (start -33.02 92.71) (end -40.64 92.71) (angle 90) (layer Edge.Cuts) (width 0.15))
   (gr_line (start -40.64 92.71) (end -25.4 69.85) (angle 90) (layer Edge.Cuts) (width 0.15))
@@
   (gr_line (start -25.4 46.99) (end -10.16 24.13) (angle 90) (layer Edge.Cuts) (width 0.15))
   (gr_line (start -10.16 24.13) (end -17.78 24.13) (angle 90) (layer Edge.Cuts) (width 0.15))
-  (gr_line (start -48.26 115.57) (end -63.5 92.71) (angle 90) (layer Edge.Cuts) (width 0.15))
   (gr_line (start -63.5 92.71) (end -55.88 92.71) (angle 90) (layer Edge.Cuts) (width 0.15))
   (gr_line (start -55.88 92.71) (end -71.12 69.85) (angle 90) (layer Edge.Cuts) (width 0.15))

Commit message: finished tree!
Parts:
- added J1: OUT1, Connectors:Pin_d0.9mm_L10.0mm_W2.4mm_FlatFork, F.Cu at (188.9, 59.8)
- added J10: VCC, Connectors:Pin_d0.9mm_L10.0mm_W2.4mm_FlatFork, F.Cu at (66.2, 67.0)
- added J2: IN1, Connectors:Pin_d0.9mm_L10.0mm_W2.4mm_FlatFork, F.Cu at (66.2, 61.3)
- added J3: OUT2, Connectors:Pin_d0.9mm_L10.0mm_W2.4mm_FlatFork, F.Cu at (66.2, 69.8)
- added J4: IN2, Connectors:Pin_d0.9mm_L10.0mm_W2.4mm_FlatFork, F.Cu at (198.2, 68.3)
- added J5: OUT3, Connectors:Pin_d0.9mm_L10.0mm_W2.4mm_FlatFork, F.Cu at (198.2, 59.8)
- added J6: IN3, Connectors:Pin_d0.9mm_L10.0mm_W2.4mm_FlatFork, F.Cu at (75.5, 61.3)
- added J7: GND, Connectors:Pin_d0.9mm_L10.0mm_W2.4mm_FlatFork, F.Cu at (188.9, 65.5)
- added J8: GND, Connectors:Pin_d0.9mm_L10.0mm_W2.4mm_FlatFork, F.Cu at (66.2, 64.1)
- added J9: VCC, Connectors:Pin_d0.9mm_L10.0mm_W2.4mm_FlatFork, F.Cu at (188.9, 62.6)
- added REF**: VIA, ledTree:VIA, F.Cu at (67.0, 86.4)
- added REF**: VIA, ledTree:VIA, F.Cu at (73.7, 86.4)
- added U1: ATTINY85, ledTree:ATTINY85, F.Cu at (166.5, 36.4)
- added U14: WS2812b, LEDs:LED_D5.0mm-4, F.Cu at (98.1, 45.2)
- added U15: WS2812b, LEDs:LED_D5.0mm-4, F.Cu at (90.5, 68.0)
- added U16: WS2812b, LEDs:LED_D5.0mm-4, F.Cu at (82.9, 90.9)
- added U17: WS2812b, LEDs:LED_D5.0mm-4, F.Cu at (75.2, 113.8)
- moved U11 280.3 mm to (213.2, 66.5), turned to 90 degrees
- moved U4 259.5 mm to (181.6, 89.4), turned to 90 degrees
- moved U2 227.5 mm to (166.3, 43.7)
- moved SW1 163.1 mm to (203.9, 38.0)
- moved U10 120.2 mm to (220.8, 43.7), turned to 90 degrees
- moved U8 113.7 mm to (58.9, 90.9)
- moved U13 96.5 mm to (197.9, 112.2), turned to 90 degrees
- moved U12 83.0 mm to (205.5, 89.4), turned to 90 degrees
- moved U5 82.2 mm to (189.2, 112.2), turned to 90 degrees
- moved U6 76.4 mm to (43.6, 45.2), turned to 90 degrees
- moved U9 67.6 mm to (66.5, 113.8), turned to 90 degrees
- moved U7 66.6 mm to (51.3, 68.0), turned to 90 degrees
- moved U3 66.5 mm to (173.9, 66.5), turned to 90 degrees
Connections:
- U10 pad 2: VCC -> GND
- U10 pad 3: GND -> VCC
- U10 pad 4: Net-(U10-Pad4) -> /IN2
- U11 pad 2: VCC -> GND
- U11 pad 3: GND -> VCC
- U11 pad 4: Net-(U11-Pad4) -> Net-(U10-Pad1)
- U12 pad 2: VCC -> GND
- U12 pad 3: GND -> VCC
- U12 pad 4: Net-(U12-Pad4) -> Net-(U11-Pad1)
- U13 pad 1: Net-(U13-Pad1) -> /OUT3
- U13 pad 2: VCC -> GND
- U13 pad 3: GND -> VCC
- U13 pad 4: Net-(U13-Pad4) -> Net-(U12-Pad1)
- U2 pad 1: Net-(U1-Pad2) -> Net-(U2-Pad1)
- U2 pad 2: VCC -> GND
- U2 pad 3: GND -> VCC
- U2 pad 4: Net-(U2-Pad4) -> Net-(U1-Pad2)
- U3 pad 1: Net-(U10-Pad4) -> Net-(U3-Pad1)
- U3 pad 2: VCC -> GND
- U3 pad 3: GND -> VCC
- U3 pad 4: Net-(U3-Pad4) -> Net-(U2-Pad1)
- U4 pad 1: Net-(U11-Pad4) -> Net-(U4-Pad1)
- U4 pad 2: VCC -> GND
- U4 pad 3: GND -> VCC
- U4 pad 4: Net-(U4-Pad4) -> Net-(U3-Pad1)
- U5 pad 1: Net-(U12-Pad4) -> /OUT1
- U5 pad 2: VCC -> GND
- U5 pad 3: GND -> VCC
- U5 pad 4: Net-(U5-Pad4) -> Net-(U4-Pad1)
- U6 pad 1: Net-(U2-Pad4) -> Net-(U6-Pad1)
- U6 pad 2: VCC -> GND
- U6 pad 3: GND -> VCC
- U6 pad 4: Net-(U10-Pad1) -> /IN1
- U7 pad 1: Net-(U3-Pad4) -> Net-(U7-Pad1)
- U7 pad 2: VCC -> GND
- U7 pad 3: GND -> VCC
- U7 pad 4: Net-(U11-Pad1) -> Net-(U6-Pad1)
- U8 pad 1: Net-(U4-Pad4) -> Net-(U8-Pad1)
- U8 pad 2: VCC -> GND
- U8 pad 3: GND -> VCC
- U8 pad 4: Net-(U12-Pad1) -> Net-(U7-Pad1)
- U9 pad 1: Net-(U5-Pad4) -> /OUT2
- U9 pad 2: VCC -> GND
- U9 pad 3: GND -> VCC
- U9 pad 4: Net-(U13-Pad1) -> Net-(U8-Pad1)
Routing:
- net /OUT1: track 0.00 -> 57.7 mm
- net /OUT3: track 0.00 -> 56.2 mm
- net /OUT2: track 0.00 -> 49.4 mm
- net /IN2: track 0.00 -> 40.3 mm
- net /IN3: track 0.00 -> 39.3 mm
- net /IN1: track 0.00 -> 34.1 mm
- net Net-(U1-Pad2): track 0.00 -> 24.2 mm
- net Net-(U2-Pad1): track 0.00 -> 22.2 mm
- net Net-(U10-Pad1): track 0.00 -> 22.2 mm
- net Net-(U7-Pad1): track 0.00 -> 22.2 mm
- net Net-(U4-Pad1): track 0.00 -> 22.2 mm
- net Net-(U14-Pad1): track 0.00 -> 22.2 mm
- net Net-(U8-Pad1): track 0.00 -> 22.2 mm
- net Net-(U3-Pad1): track 0.00 -> 22.2 mm
- net Net-(U15-Pad1): track 0.00 -> 22.2 mm
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- added copper zone on F.Cu, net GND
- added copper zone on B.Cu, net VCC
Other:
- board size 124.5 x 115.1 mm -> 198.9 x 100 mm

Commit message: update
Parts:
- J7: value GND -> VCC
- J9: value VCC -> GND
- moved J9 0.14 mm to (189.0, 62.7), turned to 0 degrees
- moved J7 0.09 mm to (189.0, 65.5), turned to 0 degrees
Connections:
- J7 pad 1: GND -> VCC
- J9 pad 1: VCC -> GND
Other:
- board text added: "IN3"
- board text added: "OUT2 VCC GND IN1"
- board text added: "OUT3 IN2"
- board text added: "VCC GND OUT1"
Changed lines of the file:
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@@
-(kicad_pcb (version 4) (host pcbnew 4.0.7-e2-6376~58~ubuntu16.04.1)
+(kicad_pcb (version 4) (host pcbnew 4.0.7)
   (general
     (links 59)
     (no_connects 2)
-    (area 23.1013 18.7325 124.371101 131.445001)
+    (area 23.1013 18.7325 245.681501 131.445001)
     (thickness 1.6)
-    (drawings 126)
+    (drawings 130)
     (tracks 68)
     (zones 0)
@@
     (mod_text_size 1 1)
     (mod_text_width 0.15)
-    (pad_size 2 2)
-    (pad_drill 1.1)
+    (pad_size 1.8 1.8)
+    (pad_drill 0.9)
     (pad_to_mask_clearance 0.2)
     (aux_axis_origin 0 0)
     (visible_elements 7FFFFFFF)
     (pcbplotparams
-      (layerselection 0x010fc_80000001)
+      (layerselection 0x00020_00000000)
       (usegerberextensions false)
-      (excludeedgelayer true)
+      (excludeedgelayer false)
       (linewidth 0.100000)
       (plotframeref false)
@@
       (padsonsilk false)
       (subtractmaskfromsilk false)
-      (outputformat 1)
+      (outputformat 4)
       (mirror false)
       (drillshape 0)
       (scaleselection 1)
-      (outputdirectory /home/rocket3989/Desktop/gerberout/))
+      (outputdirectory C:/Users/rocket3989/Desktop/))
   )
   (net 0 "")
@@
     (descr "solder Pin_ with flat fork, hole diameter 0.9mm, length 10.0mm, width 2.4mm")
     (tags "solder Pin_ with flat fork")
-    (fp_text reference J1 (at 0 1.95) (layer F.SilkS)
+    (fp_text reference J1 (at 0 1.95) (layer F.SilkS) hide
       (effects (font (size 1 1) (thickness 0.15)))
     )
@@
     (descr "solder Pin_ with flat fork, hole diameter 0.9mm, length 10.0mm, width 2.4mm")
     (tags "solder Pin_ with flat fork")
-    (fp_text reference J4 (at 0 1.95) (layer F.SilkS)
+    (fp_text reference J4 (at 0 1.95) (layer F.SilkS) hide
       (effects (font (size 1 1) (thickness 0.15)))
     )
@@
     (descr "solder Pin_ with flat fork, hole diameter 0.9mm, length 10.0mm, width 2.4mm")
     (tags "solder Pin_ with flat fork")
-    (fp_text reference J5 (at 0 1.95) (layer F.SilkS)
+    (fp_text reference J5 (at 0 1.95) (layer F.SilkS) hide
       (effects (font (size 1 1) (thickness 0.15)))
     )
@@
   )
   (module Connectors:Pin_d0.9mm_L10.0mm_W2.4mm_FlatFork (layer F.Cu)
-    (at 188.9252 65.4558 90)
+    (at 188.976 65.532)
     (descr "solder Pin_ with flat fork, hole diameter 0.9mm, length 10.0mm, width 2.4mm")
     (tags "solder Pin_ with flat fork")
-    (fp_text reference J7 (at 0 1.95 90) (layer F.SilkS)
-      (effects (font (size 1 1) (thickness 0.15)))
-    )
-    (fp_text value GND (at 0 -2.05 90) (layer F.Fab)
-      (effects (font (size 1 1) (thickness 0.15)))
-    )
-    (fp_text user %R (at 0 1.95 90) (layer F.Fab)
+    (fp_text reference J7 (at 0 1.95) (layer F.SilkS) hide
+      (effects (font (size 1 1) (thickness 0.15)))
+    )
+    (fp_text value VCC (at 0 -2.05) (layer F.Fab)
+      (effects (font (size 1 1) (thickness 0.15)))
+    )
+    (fp_text user %R (at 0 1.95) (layer F.Fab)
       (effects (font (size 1 1) (thickness 0.15)))
     )
@@
     (fp_line (start 1.7 1.4) (end 1.7 -1.4) (layer F.CrtYd) (width 0.05))
     (fp_line (start 1.7 1.4) (end -1.7 1.4) (layer F.CrtYd) (width 0.05))
-    (pad 1 thru_hole circle (at 0 0 90) (size 1.8 1.8) (drill 0.9) (layers *.Cu *.Mask)
-      (net 2 GND))
+    (pad 1 thru_hole circle (at 0 0) (size 1.8 1.8) (drill 0.9) (layers *.Cu *.Mask)
+      (net 4 VCC))
     (model ${KISYS3DMOD}/Connectors.3dshapes/Pin_d0.9mm_L10.0mm_W2.4mm_FlatFork.wrl
       (at (xyz 0 0 0))
@@
   )
   (module Connectors:Pin_d0.9mm_L10.0mm_W2.4mm_FlatFork (layer F.Cu)
-    (at 188.9252 62.611 90)
+    (at 188.976 62.738)
     (descr "solder Pin_ with flat fork, hole diameter 0.9mm, length 10.0mm, width 2.4mm")
     (tags "solder Pin_ with flat fork")
-    (fp_text reference J9 (at 0 1.95 90) (layer F.SilkS)
-      (effects (font (size 1 1) (thickness 0.15)))
-    )
-    (fp_text value VCC (at 0 -2.05 90) (layer F.Fab)
-      (effects (font (size 1 1) (thickness 0.15)))
-    )
-    (fp_text user %R (at 0 1.95 90) (layer F.Fab)
+    (fp_text reference J9 (at 0 1.95) (layer F.SilkS) hide
+      (effects (font (size 1 1) (thickness 0.15)))
+    )
+    (fp_text value GND (at 0 -2.05) (layer F.Fab)
+      (effects (font (size 1 1) (thickness 0.15)))
+    )
+    (fp_text user %R (at 0 1.95) (layer F.Fab)
       (effects (font (size 1 1) (thickness 0.15)))
     )
@@
     (fp_line (start 1.7 1.4) (end 1.7 -1.4) (layer F.CrtYd) (width 0.05))
     (fp_line (start 1.7 1.4) (end -1.7 1.4) (layer F.CrtYd) (width 0.05))
-    (pad 1 thru_hole circle (at 0 0 90) (size 1.8 1.8) (drill 0.9) (layers *.Cu *.Mask)
-      (net 4 VCC))
+    (pad 1 thru_hole circle (at 0 0) (size 1.8 1.8) (drill 0.9) (layers *.Cu *.Mask)
+      (net 2 GND))
     (model ${KISYS3DMOD}/Connectors.3dshapes/Pin_d0.9mm_L10.0mm_W2.4mm_FlatFork.wrl
       (at (xyz 0 0 0))
@@
     (descr "solder Pin_ with flat fork, hole diameter 0.9mm, length 10.0mm, width 2.4mm")
     (tags "solder Pin_ with flat fork")
-    (fp_text reference J2 (at 0 1.95) (layer F.SilkS)
+    (fp_text reference J2 (at 0 1.95) (layer F.SilkS) hide
       (effects (font (size 1 1) (thickness 0.15)))
     )
@@
     (descr "solder Pin_ with flat fork, hole diameter 0.9mm, length 10.0mm, width 2.4mm")
     (tags "solder Pin_ with flat fork")
-    (fp_text reference J3 (at 0 1.95) (layer F.SilkS)
+    (fp_text reference J3 (at 0 1.95) (layer F.SilkS) hide
       (effects (font (size 1 1) (thickness 0.15)))
     )
@@
     (descr "solder Pin_ with flat fork, hole diameter 0.9mm, length 10.0mm, width 2.4mm")
     (tags "solder Pin_ with flat fork")
-    (fp_text reference J6 (at 0 1.95) (layer F.SilkS)
+    (fp_text reference J6 (at 0 1.95) (layer F.SilkS) hide
       (effects (font (size 1 1) (thickness 0.15)))
     )
@@
     (descr "solder Pin_ with flat fork, hole diameter 0.9mm, length 10.0mm, width 2.4mm")
     (tags "solder Pin_ with flat fork")
-    (fp_text reference J8 (at 0 1.95) (layer F.SilkS)
+    (fp_text reference J8 (at 0 1.95) (layer F.SilkS) hide
       (effects (font (size 1 1) (thickness 0.15)))
     )
@@
     (descr "solder Pin_ with flat fork, hole diameter 0.9mm, length 10.0mm, width 2.4mm")
     (tags "solder Pin_ with flat fork")
-    (fp_text reference J10 (at 0 1.95) (layer F.SilkS)
+    (fp_text reference J10 (at 0 1.95) (layer F.SilkS) hide
       (effects (font (size 1 1) (thickness 0.15)))
     )
@@
       (net 2 GND))
   )
+  (gr_text IN3 (at 77.978 61.214 270) (layer F.SilkS)
+    (effects (font (size 0.762 0.762) (thickness 0.1905)))
+  )
+  (gr_text "OUT3            IN2" (at 200.914 63.754 270) (layer F.SilkS)
+    (effects (font (size 0.762 0.762) (thickness 0.1905)))
+  )
+  (gr_text "VCC GND OUT1\n" (at 186.436 62.484 90) (layer F.SilkS)
+    (effects (font (size 0.762 0.762) (thickness 0.1905)))
+  )
+  (gr_text "OUT2 VCC GND IN1" (at 63.5 65.786 90) (layer F.SilkS)
+    (effects (font (size 0.762 0.762) (thickness 0.1905)))
+  )
   (gr_line (start 208.788 81.407) (end 218.3638 67.0052) (angle 90) (layer Edge.Cuts) (width 0.01))

Commit message: update
Parts:
- added C1: CP, Capacitors_THT:CP_Radial_D5.0mm_P2.50mm, F.Cu at (176.9, 57.2)
- added RV1: POT, Potentiometers:Potentiometer_Trimmer_Bourns_3339S_Vertical, F.Cu at (182.2, 74.7)
- J7: value VCC -> GND
- J9: value GND -> VCC
Connections:
- J7 pad 1: VCC -> GND
- J9 pad 1: GND -> VCC
- U1 pad 2: Net-(U1-Pad2) -> Net-(RV1-Pad2)
- U2 pad 4: Net-(U1-Pad2) -> Net-(U1-Pad0)
Routing:
- net Net-(RV1-Pad2): track 0.00 -> 31.1 mm
- net Net-(U1-Pad0): track 0.00 -> 26.3 mm
- net Net-(U1-Pad2): track 24.2 -> 0.00 mm
- net /OUT3: track 56.2 -> 57.4 mm
- net /OUT1: track 57.7 -> 56.9 mm
- net /IN2: track 40.3 -> 41.1 mm
