File: ledTree/ledTree.kicad_pcb (KiCad board)
At the start: 2 copper layers, 198.9 x 100 mm, 32 parts, among them J1 OUT1, J10 VCC, J2 IN1, J3 OUT2, J4 IN2, J5 OUT3, J6 IN3, J7 GND, J8 GND, J9 VCC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

Commit message: updates
Parts:
- moved J7 2.92 mm to (188.9, 62.6)
- moved J9 2.72 mm to (188.9, 65.5)
Connections:
- U1 pad 1: Net-(U1-Pad1) -> Net-(SW1-Pad2)
- U1 pad 5: Net-(SW1-Pad2) -> Net-(U1-Pad5)
Changed lines of the file:
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@@
   )
   (setup
-    (last_trace_width 0.25)
+    (last_trace_width 0.5)
     (user_trace_width 0.5)
     (trace_clearance 0.2)
@@
     (mod_text_size 1 1)
     (mod_text_width 0.15)
-    (pad_size 1.8 1.8)
-    (pad_drill 0.9)
+    (pad_size 2 2)
+    (pad_drill 1.1)
     (pad_to_mask_clearance 0.2)
     (aux_axis_origin 0 0)
@@
   (net 23 "Net-(U1-Pad4)")
   (net 24 "Net-(U1-Pad3)")
-  (net 25 "Net-(U1-Pad1)")
-  (net 26 "Net-(U1-Pad0)")
-  (net 27 "Net-(U1-Pad8)")
-  (net 28 "Net-(RV1-Pad2)")
+  (net 25 "Net-(U1-Pad0)")
+  (net 26 "Net-(U1-Pad8)")
+  (net 27 "Net-(RV1-Pad2)")
+  (net 28 "Net-(U1-Pad5)")
   (net_class Default "This is the default net class."
     (clearance 0.2)
@@
     (add_net "Net-(SW1-Pad2)")
     (add_net "Net-(U1-Pad0)")
-    (add_net "Net-(U1-Pad1)")
     (add_net "Net-(U1-Pad3)")
     (add_net "Net-(U1-Pad4)")
+    (add_net "Net-(U1-Pad5)")
     (add_net "Net-(U1-Pad8)")
     (add_net "Net-(U10-Pad1)")
@@
       (net 3 VCC))
     (pad 4 thru_hole oval (at 3.81 0 90) (size 1.07 1.8) (drill 0.9) (layers *.Cu *.Mask)
-      (net 26 "Net-(U1-Pad0)"))
+      (net 25 "Net-(U1-Pad0)"))
     (model ${KISYS3DMOD}/LEDs.3dshapes/LED_D5.0mm-4.wrl
       (at (xyz 0 0 0))
@@
     (fp_line (start 4 17.5) (end 4 0) (layer F.SilkS) (width 0.15))
     (pad 5 thru_hole circle (at 21.82 1.04) (size 1.524 1.524) (drill 0.762) (layers *.Cu *.Mask)
-      (net 1 "Net-(SW1-Pad2)"))
+      (net 28 "Net-(U1-Pad5)"))
     (pad 4 thru_hole circle (at 21.82 3.58) (size 1.524 1.524) (drill 0.762) (layers *.Cu *.Mask)
       (net 23 "Net-(U1-Pad4)"))
@@
       (net 24 "Net-(U1-Pad3)"))
     (pad 2 thru_hole circle (at 21.82 8.66) (size 1.524 1.524) (drill 0.762) (layers *.Cu *.Mask)
-      (net 28 "Net-(RV1-Pad2)"))
+      (net 27 "Net-(RV1-Pad2)"))
     (pad 1 thru_hole circle (at 21.82 11.2) (size 1.524 1.524) (drill 0.762) (layers *.Cu *.Mask)
-      (net 25 "Net-(U1-Pad1)"))
+      (net 1 "Net-(SW1-Pad2)"))
     (pad 0 thru_hole circle (at 21.82 13.74) (size 1.524 1.524) (drill 0.762) (layers *.Cu *.Mask)
-      (net 26 "Net-(U1-Pad0)"))
+      (net 25 "Net-(U1-Pad0)"))
     (pad 8 thru_hole circle (at 14.2 16.28) (size 1.524 1.524) (drill 0.762) (layers *.Cu *.Mask)
-      (net 27 "Net-(U1-Pad8)"))
+      (net 26 "Net-(U1-Pad8)"))
     (pad 7 thru_hole circle (at 11.66 16.28) (size 1.524 1.524) (drill 0.762) (layers *.Cu *.Mask)
       (net 2 GND))
@@
   )
   (module Connectors:Pin_d0.9mm_L10.0mm_W2.4mm_FlatFork (layer F.Cu)
-    (at 188.976 65.532)
+    (at 188.9252 62.611)
     (descr "solder Pin_ with flat fork, hole diameter 0.9mm, length 10.0mm, width 2.4mm")
     (tags "solder Pin_ with flat fork")
@@
   )
   (module Connectors:Pin_d0.9mm_L10.0mm_W2.4mm_FlatFork (layer F.Cu)
-    (at 188.976 62.738)
+    (at 188.9252 65.4558)
     (descr "solder Pin_ with flat fork, hole diameter 0.9mm, length 10.0mm, width 2.4mm")
     (tags "solder Pin_ with flat fork")
@@
       (net 3 VCC))
     (pad 2 thru_hole circle (at -2.54 2.54 180) (size 1.44 1.44) (drill 0.8) (layers *.Cu *.Mask)
-      (net 28 "Net-(RV1-Pad2)"))
+      (net 27 "Net-(RV1-Pad2)"))
     (pad 1 thru_hole circle (at 0 0 180) (size 1.44 1.44) (drill 0.8) (layers *.Cu *.Mask)
       (net 2 GND))
@@
   (gr_line (start 99.2632 63.1952) (end 91.7448 63.1952) (angle 90) (layer Edge.Cuts) (width 0.01))
   (gr_line (start 86.106 82.931) (end 95.6818 68.5292) (angle 90) (layer Edge.Cuts) (width 0.01))
-  (segment (start 188.3424 37.4382) (end 198.8637 37.4382) (width 0.25) (layer F.Cu) (net 1))
-  (segment (start 198.8637 37.4382) (end 203.9112 42.4857) (width 0.25) (layer F.Cu) (net 1))
+  (segment (start 188.3424 47.5982) (end 198.7987 47.5982) (width 0.5) (layer F.Cu) (net 1))
+  (segment (start 198.7987 47.5982) (end 203.9112 42.4857) (width 0.5) (layer F.Cu) (net 1))
   (segment (start 73.6854 86.4108) (end 67.0687 86.4108) (width 0.5) (layer B.Cu) (net 2))
   (segment (start 67.0687 86.4108) (end 67.0433 86.4362) (width 0.5) (layer B.Cu) (net 2))
@@
   (segment (start 205.5368 95.8342) (end 205.5368 89.3826) (width 0.25) (layer B.Cu) (net 6))
   (segment (start 197.9168 103.4542) (end 205.5368 95.8342) (width 0.25) (layer B.Cu) (net 6))
-  (segment (start 189.1792 112.2426) (end 190.9318 112.2426) (width 0.25) (layer B.Cu) (net 7) (status 400000))
-  (segment (start 190.9826 59.7662) (end 188.9252 59.7662) (width 0.25) (layer B.Cu) (net 7) (status 800000))
+  (segment (start 189.1792 112.2426) (end 190.9318 112.2426) (width 0.25) (layer B.Cu) (net 7))
+  (segment (start 190.9826 59.7662) (end 188.9252 59.7662) (width 0.25) (layer B.Cu) (net 7))
   (segment (start 191.643 60.4266) (end 190.9826 59.7662) (width 0.25) (layer B.Cu) (net 7))
   (segment (start 191.643 111.5314) (end 191.643 60.4266) (width 0.25) (layer B.Cu) (net 7))
@@
   (segment (start 70.7644 112.6109) (end 70.7644 82.4738) (width 0.25) (layer F.Cu) (net 9))
   (segment (start 69.6087 113.7666) (end 70.7644 112.6109) (width 0.25) (layer F.Cu) (net 9))
-  (segment (start 198.1708 68.3006) (end 199.39 68.3006) (width 0.25) (layer B.Cu) (net 10) (status 400000))
-  (segment (start 216.4588 39.8526) (end 220.7768 39.8526) (width 0.25) (layer B.Cu) (net 10) (status 800000))
+  (segment (start 198.1708 68.3006) (end 199.39 68.3006) (width 0.25) (layer B.Cu) (net 10))
+  (segment (start 216.4588 39.8526) (end 220.7768 39.8526) (width 0.25) (layer B.Cu) (net 10))
   (segment (start 207.5942 48.7172) (end 216.4588 39.8526) (width 0.25) (layer B.Cu) (net 10))
   (segment (start 207.5942 60.0964) (end 207.5942 48.7172) (width 0.25) (layer B.Cu) (net 10))
   (segment (start 199.39 68.3006) (end 207.5942 60.0964) (width 0.25) (layer B.Cu) (net 10))
-  (segment (start 197.9168 112.2426) (end 196.1642 112.2426) (width 0.25) (layer B.Cu) (net 11) (status 400000))
-  (segment (start 193.3702 64.5668) (end 198.1708 59.7662) (width 0.25) (layer B.Cu) (net 11) (status 800000))
+  (segment (start 197.9168 112.2426) (end 196.1642 112.2426) (width 0.25) (layer B.Cu) (net 11))
+  (segment (start 193.3702 64.5668) (end 198.1708 59.7662) (width 0.25) (layer B.Cu) (net 11))
   (segment (start 193.3702 69.977) (end 193.3702 64.5668) (width 0.25) (layer B.Cu) (net 11))
   (segment (start 195.199 71.8058) (end 193.3702 69.977) (width 0.25) (layer B.Cu) (net 11))
@@
   (segment (start 75.2348 99.6696) (end 75.2348 109.9566) (width 0.25) (layer B.Cu) (net 21))
   (segment (start 82.8548 92.0496) (end 75.2348 99.6696) (width 0.25) (layer B.Cu) (net 21))
-  (segment (start 188.3424 50.1382) (end 183.3104 50.1382) (width 0.25) (layer B.Cu) (net 26))
-  (segment (start 173.0248 39.8526) (end 166.3192 39.8526) (width 0.25) (layer B.Cu) (net 26))
-  (segment (start 183.3104 50.1382) (end 173.0248 39.8526) (width 0.25) (layer B.Cu) (net 26))
-  (segment (start 184.7596 72.1614) (end 184.7596 66.8528) (width 0.25) (layer B.Cu) (net 28) (status 400000))
-  (segment (start 190.6016 47.3174) (end 188.3424 45.0582) (width 0.25) (layer B.Cu) (net 28) (status 800000))
-  (segment (start 190.6016 51.4096) (end 190.6016 47.3174) (width 0.25) (layer B.Cu) (net 28))
-  (segment (start 183.9468 58.0644) (end 190.6016 51.4096) (width 0.25) (layer B.Cu) (net 28))
-  (segment (start 183.9468 66.04) (end 183.9468 58.0644) (width 0.25) (layer B.Cu) (net 28))
-  (segment (start 184.7596 66.8528) (end 183.9468 66.04) (width 0.25) (layer B.Cu) (net 28))
+  (segment (start 188.3424 50.1382) (end 183.3104 50.1382) (width 0.25) (layer B.Cu) (net 25))
+  (segment (start 173.0248 39.8526) (end 166.3192 39.8526) (width 0.25) (layer B.Cu) (net 25))
+  (segment (start 183.3104 50.1382) (end 173.0248 39.8526) (width 0.25) (layer B.Cu) (net 25))
+  (segment (start 184.7596 72.1614) (end 184.7596 66.8528) (width 0.25) (layer B.Cu) (net 27))
+  (segment (start 190.6016 47.3174) (end 188.3424 45.0582) (width 0.25) (layer B.Cu) (net 27))
+  (segment (start 190.6016 51.4096) (end 190.6016 47.3174) (width 0.25) (layer B.Cu) (net 27))
+  (segment (start 183.9468 58.0644) (end 190.6016 51.4096) (width 0.25) (layer B.Cu) (net 27))
+  (segment (start 183.9468 66.04) (end 183.9468 58.0644) (width 0.25) (layer B.Cu) (net 27))
+  (segment (start 184.7596 66.8528) (end 183.9468 66.04) (width 0.25) (layer B.Cu) (net 27))
   (zone (net 3) (net_name VCC) (layer B.Cu) (hatch edge 0.508)
     (connect_pads (clearance 0.508))
