File: 555 pwm/555 pwm.kicad_pcb (KiCad board)
At the start: 2 copper layers, 46.9 x 19.8 mm, 12 parts, among them M1 Motor_DC, Q1 PN2222A, U1 NE555

Commit message: many updates
Parts:
- added SW1: SW_DIP_x01, Connectors:Wafer_Vertical10x5.8x7RM2.5-3, F.Cu at (127.5, 87.9)
- Q1: footprint TO_SOT_Packages_THT:TO-92_Molded_Wide -> TO_SOT_Packages_THT:TO-92_Inline_Wide
- moved C1 4.64 mm to (118.7, 84.7)
- moved RV1 2.22 mm to (144.7, 85.1)
- moved BT1 0.93 mm to (132.1, 88.1), turned to 0 degrees
- moved Q1 0.23 mm to (103.9, 73.6)
- moved D3 0.18 mm to (107.7, 89.6)
Connections:
- D3 pad 1: Net-(BT1-Pad1) -> Net-(D3-Pad1)
- M1 pad 1: Net-(BT1-Pad1) -> Net-(D3-Pad1)
- R2 pad 2: Net-(BT1-Pad1) -> Net-(D3-Pad1)
- U1 pad 4: Net-(BT1-Pad1) -> Net-(D3-Pad1)
- U1 pad 8: Net-(BT1-Pad1) -> Net-(D3-Pad1)
Routing:
- net Net-(C2-Pad1): track 21.5 -> 43.8 mm
- net Net-(BT1-Pad1): track 0.00 -> 9.45 mm
- net Net-(D2-Pad2): track 0.00 -> 8.81 mm
- net Net-(D1-Pad1): track 0.71 -> 8.90 mm
- net Net-(Q1-Pad2): track 6.79 -> 9.43 mm
- net Net-(C1-Pad1): track 4.95 -> 6.14 mm
- added copper zone on F.Cu, net Net-(D3-Pad1)
- removed copper zone on F.Cu, net Net-(BT1-Pad1)
Other:
- board size 46.9 x 19.8 mm -> 45.7 x 19.8 mm

Commit message: updates
Parts:
- renumbered BT1 to BAT, M1 to MOTOR, RV1 to POT, SW1 to SWITCH, Q1 to TRANS
Changed lines of the file:
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@@
-(kicad_pcb (version 4) (host pcbnew 4.0.7-e2-6376~58~ubuntu16.04.1)
+(kicad_pcb (version 4) (host pcbnew 4.0.7)
   (general
     (links 23)
     (no_connects 0)
-    (area 100.483599 70.943399 146.379001 90.930801)
+    (area 93.9546 53.721 168.808401 94.716601)
     (thickness 1.6)
     (drawings 4)
@@
     (pad_to_mask_clearance 0.2)
     (aux_axis_origin 0 0)
-    (visible_elements FFFFFF7F)
+    (visible_elements 7FFFFFFF)
     (pcbplotparams
-      (layerselection 0x00030_80000001)
+      (layerselection 0x010f0_80000001)
       (usegerberextensions false)
       (excludeedgelayer true)
@@
       (drillshape 0)
       (scaleselection 1)
-      (outputdirectory ""))
+      (outputdirectory gerber/))
   )
   (net 0 "")
@@
     (descr "8-lead though-hole mounted DIP package, row spacing 7.62 mm (300 mils), Socket")
     (tags "THT DIP DIL PDIP 2.54mm 7.62mm 300mil Socket")
-    (fp_text reference U1 (at 3.81 -2.33) (layer F.SilkS)
+    (fp_text reference U1 (at 3.7846 3.81) (layer F.SilkS)
       (effects (font (size 1 1) (thickness 0.15)))
     )
@@
     (descr "C, Disc series, Radial, pin pitch=2.50mm, , diameter*width=3.8*2.6mm^2, Capacitor, http://www.vishay.com/docs/45233/krseries.pdf")
     (tags "C Disc series Radial pin pitch 2.50mm  diameter 3.8mm width 2.6mm Capacitor")
-    (fp_text reference C1 (at 1.25 -2.61 270) (layer F.SilkS)
+    (fp_text reference C1 (at 4.3434 0.0762 270) (layer F.SilkS)
       (effects (font (size 1 1) (thickness 0.15)))
     )
@@
     (descr "CP, Radial series, Radial, pin pitch=2.50mm, , diameter=5mm, Electrolytic Capacitor")
     (tags "CP Radial series Radial pin pitch 2.50mm  diameter 5mm Electrolytic Capacitor")
-    (fp_text reference C2 (at 1.25 -3.81 270) (layer F.SilkS)
+    (fp_text reference C2 (at 4.2672 -2.4384 270) (layer F.SilkS)
       (effects (font (size 1 1) (thickness 0.15)))
     )
@@
     (descr "simple 2-pin terminal block, pitch 5.08mm, revamped version of bornier2")
     (tags "terminal block bornier2")
-    (fp_text reference M1 (at 2.54 -5.08 90) (layer F.SilkS)
+    (fp_text reference MOTOR (at 2.921 2.54 90) (layer F.SilkS)
       (effects (font (size 1 1) (thickness 0.15)))
     )
@@
     (descr "Resistor, Axial_DIN0207 series, Axial, Horizontal, pin pitch=7.62mm, 0.25W = 1/4W, length*diameter=6.3*2.5mm^2, http://cdn-reichelt.de/documents/datenblatt/B400/1_4W%23YAG.pdf")
     (tags "Resistor Axial_DIN0207 series Axial Horizontal pin pitch 7.62mm 0.25W = 1/4W length 6.3mm diameter 2.5mm")
-    (fp_text reference R1 (at 3.81 -2.31 90) (layer F.SilkS)
+    (fp_text reference R1 (at 3.937 0 90) (layer F.SilkS)
       (effects (font (size 1 1) (thickness 0.15)))
     )
@@
     (descr "Resistor, Axial_DIN0207 series, Axial, Horizontal, pin pitch=7.62mm, 0.25W = 1/4W, length*diameter=6.3*2.5mm^2, http://cdn-reichelt.de/documents/datenblatt/B400/1_4W%23YAG.pdf")
     (tags "Resistor Axial_DIN0207 series Axial Horizontal pin pitch 7.62mm 0.25W = 1/4W length 6.3mm diameter 2.5mm")
-    (fp_text reference R2 (at 3.81 -2.31 180) (layer F.SilkS)
+    (fp_text reference R2 (at 3.7592 0.0508 180) (layer F.SilkS)
       (effects (font (size 1 1) (thickness 0.15)))
     )
@@
     (descr "Potentiometer, vertically mounted, Omeg PC16PU, Omeg PC16PU, Omeg PC16PU, Vishay/Spectrol 248GJ/249GJ Single, Vishay/Spectrol 248GJ/249GJ Single, Vishay/Spectrol 248GJ/249GJ Single, Vishay/Spectrol 248GH/249GH Single, Vishay/Spectrol 148/149 Single, Vishay/Spectrol 148/149 Single, Vishay/Spectrol 148/149 Single, Vishay/Spectrol 148A/149A Single with mounting plates, Vishay/Spectrol 148/149 Double, Vishay/Spectrol 148A/149A Double with mounting plates, Piher PC-16 Single, Piher PC-16 Single, Piher PC-16 Single, Piher PC-16SV Single, Piher PC-16 Double, Piher PC-16 Triple, Piher T16H Single, Piher T16L Single, Piher T16H Double, Alps RK163 Single, http://www.alps.com/prod/info/E/PDF/Potentiometer/MetalShaft/RK163/RK163.PDF")
     (tags "Potentiometer vertical  Omeg PC16PU  Omeg PC16PU  Omeg PC16PU  Vishay/Spectrol 248GJ/249GJ Single  Vishay/Spectrol 248GJ/249GJ Single  Vishay/Spectrol 248GJ/249GJ Single  Vishay/Spectrol 248GH/249GH Single  Vishay/Spectrol 148/149 Single  Vishay/Spectrol 148/149 Single  Vishay/Spectrol 148/149 Single  Vishay/Spectrol 148A/149A Single with mounting plates  Vishay/Spectrol 148/149 Double  Vishay/Spectrol 148A/149A Double with mounting plates  Piher PC-16 Single  Piher PC-16 Single  Piher PC-16 Single  Piher PC-16SV Single  Piher PC-16 Double  Piher PC-16 Triple  Piher T16H Single  Piher T16L Single  Piher T16H Double  Alps RK163 Single")
-    (fp_text reference RV1 (at 0 -15.2) (layer F.SilkS)
+    (fp_text reference POT (at -3.2004 -5.1054 90) (layer F.SilkS)
       (effects (font (size 1 1) (thickness 0.15)))
     )
@@
     (descr "D, A-405 series, Axial, Horizontal, pin pitch=10.16mm, , length*diameter=5.2*2.7mm^2, , http://www.diodes.com/_files/packages/A-405.pdf")
     (tags "D A-405 series Axial Horizontal pin pitch 10.16mm  length 5.2mm diameter 2.7mm")
-    (fp_text reference D1 (at 5.08 -2.41 180) (layer F.SilkS)
+    (fp_text reference D1 (at 5.0546 -0.0508 180) (layer F.SilkS)
       (effects (font (size 1 1) (thickness 0.15)))
     )
@@
     (descr "D, A-405 series, Axial, Horizontal, pin pitch=10.16mm, , length*diameter=5.2*2.7mm^2, , http://www.diodes.com/_files/packages/A-405.pdf")
     (tags "D A-405 series Axial Horizontal pin pitch 10.16mm  length 5.2mm diameter 2.7mm")
-    (fp_text reference D2 (at 5.08 -2.41) (layer F.SilkS)
+    (fp_text reference D2 (at 5.1054 0.0508) (layer F.SilkS)
       (effects (font (size 1 1) (thickness 0.15)))
     )
@@
     (descr "D, A-405 series, Axial, Horizontal, pin pitch=10.16mm, , length*diameter=5.2*2.7mm^2, , http://www.diodes.com/_files/packages/A-405.pdf")
     (tags "D A-405 series Axial Horizontal pin pitch 10.16mm  length 5.2mm diameter 2.7mm")
-    (fp_text reference D3 (at 5.08 -2.41 90) (layer F.SilkS)
+    (fp_text reference D3 (at 5.1054 -0.0254 90) (layer F.SilkS)
       (effects (font (size 1 1) (thickness 0.15)))
     )
@@
     (descr GTK2400-V2)
     (tags GTK2400-V2)
-    (fp_text reference BT1 (at -3.55 -0.05 270) (layer F.SilkS)
+    (fp_text reference BAT (at 1.905 -2.2352) (layer F.SilkS)
       (effects (font (size 1 1) (thickness 0.15)))
     )
@@
     (descr "Gold-Tek vertical wafer connector with 2.5mm pitch")
     (tags "wafer connector vertical")
-    (fp_text reference SW1 (at 2.54 -3.81 180) (layer F.SilkS)
+    (fp_text reference SWITCH (at 2.54 1.9304 180) (layer F.SilkS)
       (effects (font (size 1 1) (thickness 0.15)))
     )
@@
     (descr "TO-92 leads in-line, wide, drill 0.8mm (see NXP sot054_po.pdf)")
     (tags "to-92 sc-43 sc-43a sot54 PA33 transistor")
-    (fp_text reference Q1 (at 2.54 -3.56 450) (layer F.SilkS)
+    (fp_text reference TRANS (at 2.6416 -1.905 270) (layer F.SilkS)
       (effects (font (size 1 1) (thickness 0.15)))
     )
@@
   (segment (start 114.8588 78.232) (end 111.379 74.7522) (width 0.25) (layer F.Cu) (net 9))
   (segment (start 111.379 74.7522) (end 111.379 73.152) (width 0.25) (layer F.Cu) (net 9))
-  (segment (start 103.886 76.0984) (end 106.7054 76.0984) (width 0.25) (layer F.Cu) (net 10) (status 400000))
-  (segment (start 106.7054 76.0984) (end 111.379 80.772) (width 0.25) (layer F.Cu) (net 10) (status 800000))
+  (segment (start 103.886 76.0984) (end 106.7054 76.0984) (width 0.25) (layer F.Cu) (net 10))
+  (segment (start 106.7054 76.0984) (end 111.379 80.772) (width 0.25) (layer F.Cu) (net 10))
   (zone (net 11) (net_name "Net-(D3-Pad1)") (layer F.Cu) (hatch edge 0.508)
     (connect_pads (clearance 0.508))
