File: diceroller/_saved_diceroller.sch (KiCad schematic (older format))
At the start: 18 parts, among them SW1 SW_DIP_x01, SW2 SW_DIP_x01

Commit message: additions
Parts:
- U1: renamed from U?; footprint Housings_DIP:DIP-8_W7.62mm -> Housings_DIP:DIP-8_W7.62mm_LongPads
Changed lines of the file:
@@
 	4050 1550 3950 1550
 $Comp
-L ATTINY85-20PU U?
+L ATTINY85-20PU U1
 U 1 1 5A715139
 P 2600 1700
-F 0 "U?" H 1450 2100 50  0000 C CNN
+F 0 "U1" H 1450 2100 50  0000 C CNN
 F 1 "ATTINY85-20PU" H 3600 1300 50  0000 C CNN
-F 2 "Housings_DIP:DIP-8_W7.62mm" H 3600 1700 50  0001 C CIN
+F 2 "Housings_DIP:DIP-8_W7.62mm_LongPads" H 3600 1700 50  0001 C CIN
 F 3 "" H 2600 1700 50  0001 C CNN
 	1    2600 1700
