File: diceroller/diceroller.kicad_pcb (KiCad board)
At the start: 2 copper layers, 30.5 x 31.5 mm, 18 parts, among them SW1 SW_DIP_x01, SW2 SW_DIP_x01, U1 ATTINY85-20PU

Commit message: updates
Parts:
- R3: moved to B.Cu
- SW2: moved to F.Cu
- moved R6 9.34 mm to (154.4, 97.0)
- moved R4 9.20 mm to (138.2, 93.9)
- moved SW2 6.48 mm to (141.6, 115.3), turned to 180 degrees
- moved SW1 0.51 mm to (141.7, 86.9)
- moved R3 0.10 mm to (137.6, 112.8)
- renumbered BT1 to BAT
Routing:
- net Net-(R4-Pad2): track 15.5 -> 6.38 mm
- net Net-(R2-Pad2): track 16.2 -> 21.3 mm
- net Net-(D6-Pad2): track 10.1 -> 7.18 mm
- net Net-(D4-Pad2): track 8.97 -> 9.73 mm
