File: 555 solder project/555 solder project.kicad_pcb (KiCad board)
At the start: 2 copper layers, 36.8 x 17.8 mm, 9 parts, among them SW1 SW_DIP_x01, U1 NE555

Commit message: updates
Parts:
- renumbered BT1 to BAT
Changed lines of the file:
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@@
-(kicad_pcb (version 4) (host pcbnew 4.0.7-e2-6376~58~ubuntu16.04.1)
+(kicad_pcb (version 4) (host pcbnew 4.0.7)
   (general
     (links 16)
     (no_connects 0)
-    (area 145.999999 104.089999 182.930001 121.970001)
+    (area 145.999999 101.922838 182.930001 121.970001)
     (thickness 1.6)
     (drawings 5)
@@
     (pad_to_mask_clearance 0)
     (aux_axis_origin 0 0)
-    (visible_elements FFFFFF7F)
+    (visible_elements 7FFFFFFF)
     (pcbplotparams
-      (layerselection 0x00030_80000001)
+      (layerselection 0x010fc_80000001)
       (usegerberextensions false)
       (excludeedgelayer true)
@@
       (outputformat 1)
       (mirror false)
-      (drillshape 1)
+      (drillshape 0)
       (scaleselection 1)
-      (outputdirectory ""))
+      (outputdirectory gerber/))
   )
   (net 0 "")
@@
     (descr "Through hole straight pin header, 1x02, 2.54mm pitch, single row")
     (tags "Through hole pin header THT 1x02 2.54mm single row")
-    (fp_text reference BT1 (at 0 -2.33 270) (layer F.SilkS)
+    (fp_text reference BAT (at -1.6256 1.27 360) (layer F.SilkS)
       (effects (font (size 1 1) (thickness 0.15)))
     )
@@
     (descr "LED, Round, FlatTop, diameter 5.0mm, 2 pins, http://www.kingbright.com/attachments/file/psearch/000/00/00/L-483GDT(Ver.15B).pdf")
     (tags "LED Round FlatTop diameter 5.0mm 2 pins")
-    (fp_text reference D1 (at 1.27 -4.01 270) (layer F.SilkS)
+    (fp_text reference D1 (at 1.397 -1.6256 270) (layer F.SilkS)
       (effects (font (size 1 1) (thickness 0.15)))
     )
@@
     (descr "Resistor, Axial_DIN0207 series, Axial, Horizontal, pin pitch=7.62mm, 0.25W = 1/4W, length*diameter=6.3*2.5mm^2, http://cdn-reichelt.de/documents/datenblatt/B400/1_4W%23YAG.pdf")
     (tags "Resistor Axial_DIN0207 series Axial Horizontal pin pitch 7.62mm 0.25W = 1/4W length 6.3mm diameter 2.5mm")
-    (fp_text reference R1 (at 3.81 -2.31 180) (layer F.SilkS)
+    (fp_text reference R1 (at 3.81 -0.127 180) (layer F.SilkS)
       (effects (font (size 1 1) (thickness 0.15)))
     )
@@
     (descr "Resistor, Axial_DIN0207 series, Axial, Horizontal, pin pitch=7.62mm, 0.25W = 1/4W, length*diameter=6.3*2.5mm^2, http://cdn-reichelt.de/documents/datenblatt/B400/1_4W%23YAG.pdf")
     (tags "Resistor Axial_DIN0207 series Axial Horizontal pin pitch 7.62mm 0.25W = 1/4W length 6.3mm diameter 2.5mm")
-    (fp_text reference R2 (at 3.81 -2.31) (layer F.SilkS)
+    (fp_text reference R2 (at 3.937 0) (layer F.SilkS)
       (effects (font (size 1 1) (thickness 0.15)))
     )
@@
     (descr "Resistor, Axial_DIN0207 series, Axial, Horizontal, pin pitch=7.62mm, 0.25W = 1/4W, length*diameter=6.3*2.5mm^2, http://cdn-reichelt.de/documents/datenblatt/B400/1_4W%23YAG.pdf")
     (tags "Resistor Axial_DIN0207 series Axial Horizontal pin pitch 7.62mm 0.25W = 1/4W length 6.3mm diameter 2.5mm")
-    (fp_text reference R3 (at 3.81 -2.31) (layer F.SilkS)
+    (fp_text reference R3 (at 3.937 0) (layer F.SilkS)
       (effects (font (size 1 1) (thickness 0.15)))
     )
@@
     (descr "8-lead though-hole mounted DIP package, row spacing 7.62 mm (300 mils), Socket")
     (tags "THT DIP DIL PDIP 2.54mm 7.62mm 300mil Socket")
-    (fp_text reference U1 (at 3.81 -2.33) (layer F.SilkS)
+    (fp_text reference U1 (at 3.81 1.397) (layer F.SilkS)
       (effects (font (size 1 1) (thickness 0.15)))
     )
@@
     (descr "Through hole straight pin header, 1x03, 2.54mm pitch, single row")
     (tags "Through hole pin header THT 1x03 2.54mm single row")
-    (fp_text reference SW1 (at 0 -2.33 270) (layer F.SilkS)
+    (fp_text reference SW1 (at 1.9304 2.6924 360) (layer F.SilkS)
       (effects (font (size 1 1) (thickness 0.15)))
     )
@@
   (gr_line (start 182.88 104.14) (end 146.05 104.14) (angle 90) (layer Edge.Cuts) (width 0.1))
   (gr_line (start 182.88 121.285) (end 182.88 104.14) (angle 90) (layer Edge.Cuts) (width 0.1))
-  (segment (start 161.8234 106.5276) (end 161.8234 106.4006) (width 0.25) (layer B.Cu) (net 1) (status C00000))
-  (segment (start 161.8234 106.4006) (end 160.4772 105.0544) (width 0.25) (layer B.Cu) (net 1) (status 400000))
+  (segment (start 161.8234 106.5276) (end 161.8234 106.4006) (width 0.25) (layer B.Cu) (net 1))
+  (segment (start 161.8234 106.4006) (end 160.4772 105.0544) (width 0.25) (layer B.Cu) (net 1))
   (segment (start 160.4772 105.0544) (end 156.2862 105.0544) (width 0.25) (layer B.Cu) (net 1))
-  (segment (start 156.2862 105.0544) (end 154.686 106.6546) (width 0.25) (layer B.Cu) (net 1) (status 800000))
-  (segment (start 168.91 118.11) (end 166.37 118.11) (width 0.25) (layer B.Cu) (net 2) (status C00000))
+  (segment (start 156.2862 105.0544) (end 154.686 106.6546) (width 0.25) (layer B.Cu) (net 1))
+  (segment (start 168.91 118.11) (end 166.37 118.11) (width 0.25) (layer B.Cu) (net 2))
   (segment (start 177.8 116.84) (end 177.8 113.03) (width 0.25) (layer B.Cu) (net 3))
   (segment (start 166.37 115.57) (end 176.53 115.57) (width 0.25) (layer B.Cu) (net 3))
@@
   (segment (start 158.75 113.03) (end 163.83 113.03) (width 0.25) (layer B.Cu) (net 3))
   (segment (start 163.83 113.03) (end 166.37 115.57) (width 0.25) (layer B.Cu) (net 3))
-  (segment (start 151.1554 112.903) (end 151.1554 114.2746) (width 0.25) (layer B.Cu) (net 4) (status 400000))
-  (segment (start 151.1554 114.2746) (end 148.59 116.84) (width 0.25) (layer B.Cu) (net 4) (status 800000))
+  (segment (start 151.1554 112.903) (end 151.1554 114.2746) (width 0.25) (layer B.Cu) (net 4))
+  (segment (start 151.1554 114.2746) (end 148.59 116.84) (width 0.25) (layer B.Cu) (net 4))
   (segment (start 156.21 116.84) (end 157.48 116.84) (width 0.25) (layer B.Cu) (net 5))
   (segment (start 157.48 116.84) (end 158.75 115.57) (width 0.25) (layer B.Cu) (net 5))
