File: led cube/led cube.kicad_pcb (KiCad board)
At the start: 2 copper layers, 68.1 x 57.9 mm, 22 parts, among them J0 Conn_01x01, J1 Conn_01x01, J2 Conn_01x01, J3 Conn_01x01, J4 Conn_01x01, J5 Conn_01x01, J6 Conn_01x01, J7 Conn_01x01, J8 Conn_01x01, Q1 PN2222A, Q2 PN2222A, Q3 PN2222A, SW1 SW_DIP_x01, SW2 SW_DIP_x01

Commit message: updates
Parts:
- renumbered A1 to ARDUINO, BT1 to BAT, Q1 to Q0, Q2 to Q1, Q3 to Q2, R1 to R0, R2 to R1, R3 to R2, SW1 to SWITCH
Changed lines of the file:
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@@
-(kicad_pcb (version 4) (host pcbnew 4.0.7-e2-6376~58~ubuntu16.04.1)
+(kicad_pcb (version 4) (host pcbnew 4.0.7)
   (general
     (links 29)
     (no_connects 1)
-    (area 20.244999 22.276999 88.467001 80.339001)
+    (area 12.192 16.256 99.568001 84.836001)
     (thickness 1.6)
     (drawings 6)
@@
     (pad_to_mask_clearance 0.2)
     (aux_axis_origin 0 0)
-    (visible_elements FFFFFF7F)
+    (visible_elements 7FFFFFFF)
     (pcbplotparams
-      (layerselection 0x00030_80000001)
+      (layerselection 0x010f0_80000001)
       (usegerberextensions false)
       (excludeedgelayer true)
@@
       (outputformat 1)
       (mirror false)
-      (drillshape 1)
+      (drillshape 0)
       (scaleselection 1)
-      (outputdirectory ""))
+      (outputdirectory gerber/))
   )
   (net 0 "")
@@
     (descr "Arduino Nano, http://www.mouser.com/pdfdocs/Gravitech_Arduino_Nano3_0.pdf")
     (tags "Arduino Nano")
-    (fp_text reference A1 (at 7.62 -5.08) (layer F.SilkS)
+    (fp_text reference ARDUINO (at 8.128 8.382 90) (layer F.SilkS)
       (effects (font (size 1 1) (thickness 0.15)))
     )
@@
   (module Connectors:PINHEAD1-2 (layer F.Cu)
     (at 72.644 75.184 180)
-    (fp_text reference BT1 (at 1.27 -3.9 180) (layer F.SilkS)
+    (fp_text reference BAT (at 1.27 -3.9 180) (layer F.SilkS)
       (effects (font (size 1 1) (thickness 0.15)))
     )
@@
     (descr "TO-92 leads in-line, wide, drill 0.8mm (see NXP sot054_po.pdf)")
     (tags "to-92 sc-43 sc-43a sot54 PA33 transistor")
-    (fp_text reference Q1 (at 2.54 -3.56 270) (layer F.SilkS)
+    (fp_text reference Q0 (at 2.667 -1.778 90) (layer F.SilkS)
       (effects (font (size 1 1) (thickness 0.15)))
     )
@@
     (descr "TO-92 leads in-line, wide, drill 0.8mm (see NXP sot054_po.pdf)")
     (tags "to-92 sc-43 sc-43a sot54 PA33 transistor")
-    (fp_text reference Q2 (at 2.54 -3.56 270) (layer F.SilkS)
+    (fp_text reference Q1 (at 2.54 -1.651 90) (layer F.SilkS)
       (effects (font (size 1 1) (thickness 0.15)))
     )
@@
     (descr "TO-92 leads in-line, wide, drill 0.8mm (see NXP sot054_po.pdf)")
     (tags "to-92 sc-43 sc-43a sot54 PA33 transistor")
-    (fp_text reference Q3 (at 2.54 -3.56 270) (layer F.SilkS)
+    (fp_text reference Q2 (at 2.667 -1.651 90) (layer F.SilkS)
       (effects (font (size 1 1) (thickness 0.15)))
     )
@@
     (descr "Resistor, Axial_DIN0207 series, Axial, Horizontal, pin pitch=7.62mm, 0.25W = 1/4W, length*diameter=6.3*2.5mm^2, http://cdn-reichelt.de/documents/datenblatt/B400/1_4W%23YAG.pdf")
     (tags "Resistor Axial_DIN0207 series Axial Horizontal pin pitch 7.62mm 0.25W = 1/4W length 6.3mm diameter 2.5mm")
-    (fp_text reference R1 (at 3.81 -2.31 90) (layer F.SilkS)
+    (fp_text reference R0 (at 3.81 0 90) (layer F.SilkS)
       (effects (font (size 1 1) (thickness 0.15)))
     )
@@
     (descr "Resistor, Axial_DIN0207 series, Axial, Horizontal, pin pitch=7.62mm, 0.25W = 1/4W, length*diameter=6.3*2.5mm^2, http://cdn-reichelt.de/documents/datenblatt/B400/1_4W%23YAG.pdf")
     (tags "Resistor Axial_DIN0207 series Axial Horizontal pin pitch 7.62mm 0.25W = 1/4W length 6.3mm diameter 2.5mm")
-    (fp_text reference R2 (at 3.81 -2.31 90) (layer F.SilkS)
+    (fp_text reference R1 (at 3.81 0 90) (layer F.SilkS)
       (effects (font (size 1 1) (thickness 0.15)))
     )
@@
     (descr "Resistor, Axial_DIN0207 series, Axial, Horizontal, pin pitch=7.62mm, 0.25W = 1/4W, length*diameter=6.3*2.5mm^2, http://cdn-reichelt.de/documents/datenblatt/B400/1_4W%23YAG.pdf")
     (tags "Resistor Axial_DIN0207 series Axial Horizontal pin pitch 7.62mm 0.25W = 1/4W length 6.3mm diameter 2.5mm")
-    (fp_text reference R3 (at 3.81 -2.31 90) (layer F.SilkS)
+    (fp_text reference R2 (at 3.81 0 90) (layer F.SilkS)
       (effects (font (size 1 1) (thickness 0.15)))
     )
@@
     (descr "Gold-Tek vertical wafer connector with 2.5mm pitch")
     (tags "wafer connector vertical")
-    (fp_text reference SW1 (at 2.54 -3.81) (layer F.SilkS)
-      (effects (font (size 1 1) (thickness 0.15)))
-    )
+    (fp_text reference SWITCH (at 2.794 2.159) (layer F.SilkS)
+      (effects (font (size 1 1) (thickness 0.15)))
+    )
