File: simonsays/simonsays.kicad_pcb (KiCad board)
At the start: 2 copper layers, 36.3 x 30.2 mm, 16 parts, among them SW1 SW_DIP_x01, SW2 SW_DIP_x01, SW3 SW_DIP_x01, SW4 SW_DIP_x01, SW5 SW_DIP_x01, U1 ATTINY85-20PU

Commit message: updatearro
Routing:
- net Net-(D4-Pad1): track 21.2 -> 23.8 mm
Changed lines of the file:
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@@
   (general
     (links 33)
-    (no_connects 1)
-    (area 133.274999 83.617999 169.747001 113.994001)
+    (no_connects 0)
+    (area 123.19 76.2 180.848001 120.523001)
     (thickness 1.6)
     (drawings 5)
-    (tracks 47)
+    (tracks 49)
     (zones 0)
     (modules 16)
@@
   (page A4)
   (layers
-    (0 F.Cu signal)
-    (31 B.Cu signal hide)
+    (0 F.Cu signal hide)
+    (31 B.Cu signal)
     (32 B.Adhes user)
     (33 F.Adhes user)
@@
     (trace_clearance 0.2)
     (zone_clearance 0.508)
-    (zone_45_only no)
+    (zone_45_only yes)
     (trace_min 0.2)
     (segment_width 0.2)
@@
     (add_net "Net-(U1-Pad1)")
   )
+  (module Connectors:Wafer_Vertical10x5.8x7RM2.5-3 (layer F.Cu)
+    (at 144.399 101.6 90)
+    (descr "Gold-Tek vertical wafer connector with 2.5mm pitch")
+    (tags "wafer connector vertical")
+    (fp_text reference SW5 (at 2.667 -1.778 90) (layer F.SilkS)
+      (effects (font (size 1 1) (thickness 0.15)))
+    )
+    (fp_text value SW_DIP_x01 (at 2.54 5.08 90) (layer F.Fab)
+      (effects (font (size 1 1) (thickness 0.15)))
+    )
+    (fp_line (start -2.75 -2.75) (end 7.85 -2.75) (layer F.CrtYd) (width 0.05))
+    (fp_line (start 7.85 -2.75) (end 7.85 3.8) (layer F.CrtYd) (width 0.05))
+    (fp_line (start 7.85 3.8) (end -2.75 3.8) (layer F.CrtYd) (width 0.05))
+    (fp_line (start -2.75 3.8) (end -2.75 -2.75) (layer F.CrtYd) (width 0.05))
+    (fp_line (start 7.62 3.43) (end -2.54 3.43) (layer F.SilkS) (width 0.12))
+    (fp_line (start -2.54 -2.41) (end 7.62 -2.41) (layer F.SilkS) (width 0.12))
+    (fp_line (start 7.62 -2.41) (end 7.62 3.43) (layer F.SilkS) (width 0.12))
+    (fp_line (start -2.54 -2.41) (end -2.54 3.43) (layer F.SilkS) (width 0.12))
+    (pad 1 thru_hole rect (at 0 0 90) (size 2 2) (drill 1.2) (layers *.Cu *.Mask)
+      (net 1 "Net-(BT1-Pad1)"))
+    (pad 2 thru_hole circle (at 2.54 0 90) (size 2 2) (drill 1.2) (layers *.Cu *.Mask)
+      (net 12 "Net-(R1-Pad1)"))
+    (pad 3 thru_hole circle (at 5.04 0 90) (size 2 2) (drill 1.2) (layers *.Cu *.Mask))
+    (model ${KISYS3DMOD}/Connectors.3dshapes/Wafer_Vertical10x5.8x7RM2.5-3.wrl
+      (at (xyz 0 0 0))
+      (scale (xyz 4 4 4))
+      (rotate (xyz 0 0 0))
+    )
+  )
   (module Housings_DIP:DIP-8_W7.62mm (layer F.Cu)
     (at 147.701 94.996)
@@
       (at (xyz 0.005 0 0))
       (scale (xyz 0.3937 0.3937 0.3937))
-      (rotate (xyz 0 0 0))
-    )
-  )
-  (module Connectors:Wafer_Vertical10x5.8x7RM2.5-3 (layer F.Cu)
-    (at 144.399 101.6 90)
-    (descr "Gold-Tek vertical wafer connector with 2.5mm pitch")
-    (tags "wafer connector vertical")
-    (fp_text reference SW5 (at 2.667 -1.778 90) (layer F.SilkS)
-      (effects (font (size 1 1) (thickness 0.15)))
-    )
-    (fp_text value SW_DIP_x01 (at 2.54 5.08 90) (layer F.Fab)
-      (effects (font (size 1 1) (thickness 0.15)))
-    )
-    (fp_line (start -2.75 -2.75) (end 7.85 -2.75) (layer F.CrtYd) (width 0.05))
-    (fp_line (start 7.85 -2.75) (end 7.85 3.8) (layer F.CrtYd) (width 0.05))
-    (fp_line (start 7.85 3.8) (end -2.75 3.8) (layer F.CrtYd) (width 0.05))
-    (fp_line (start -2.75 3.8) (end -2.75 -2.75) (layer F.CrtYd) (width 0.05))
-    (fp_line (start 7.62 3.43) (end -2.54 3.43) (layer F.SilkS) (width 0.12))
-    (fp_line (start -2.54 -2.41) (end 7.62 -2.41) (layer F.SilkS) (width 0.12))
-    (fp_line (start 7.62 -2.41) (end 7.62 3.43) (layer F.SilkS) (width 0.12))
-    (fp_line (start -2.54 -2.41) (end -2.54 3.43) (layer F.SilkS) (width 0.12))
-    (pad 1 thru_hole rect (at 0 0 90) (size 2 2) (drill 1.2) (layers *.Cu *.Mask)
-      (net 1 "Net-(BT1-Pad1)"))
-    (pad 2 thru_hole circle (at 2.54 0 90) (size 2 2) (drill 1.2) (layers *.Cu *.Mask)
-      (net 12 "Net-(R1-Pad1)"))
-    (pad 3 thru_hole circle (at 5.04 0 90) (size 2 2) (drill 1.2) (layers *.Cu *.Mask))
-    (model ${KISYS3DMOD}/Connectors.3dshapes/Wafer_Vertical10x5.8x7RM2.5-3.wrl
-      (at (xyz 0 0 0))
-      (scale (xyz 4 4 4))
       (rotate (xyz 0 0 0))
     )
@@
   (segment (start 155.321 107.696) (end 155.321 108.458) (width 0.25) (layer F.Cu) (net 8))
   (segment (start 155.321 108.458) (end 151.13 112.649) (width 0.25) (layer F.Cu) (net 8))
+  (segment (start 145.161 107.696) (end 145.288 107.696) (width 0.25) (layer B.Cu) (net 9))
+  (segment (start 145.288 107.696) (end 149.225 103.759) (width 0.25) (layer B.Cu) (net 9))
+  (segment (start 149.225 99.06) (end 147.701 97.536) (width 0.25) (layer B.Cu) (net 9))
+  (segment (start 149.225 103.759) (end 149.225 99.06) (width 0.25) (layer B.Cu) (net 9))
   (segment (start 141.628 107.696) (end 145.161 107.696) (width 0.25) (layer F.Cu) (net 9))
   (segment (start 141.628 107.696) (end 135.128 107.696) (width 0.25) (layer F.Cu) (net 9))
   (segment (start 147.701 97.536) (end 147.701 97.663) (width 0.25) (layer B.Cu) (net 9))
-  (segment (start 147.701 97.663) (end 145.923 99.441) (width 0.25) (layer B.Cu) (net 9))
-  (segment (start 145.923 99.441) (end 145.923 106.934) (width 0.25) (layer B.Cu) (net 9))
   (segment (start 145.923 106.934) (end 145.161 107.696) (width 0.25) (layer B.Cu) (net 9))
   (segment (start 141.986 104.521) (end 136.271 104.521) (width 0.25) (layer B.Cu) (net 10))
+  (segment (start 136.271 104.521) (end 133.731 107.061) (width 0.25) (layer B.Cu) (net 10))
+  (segment (start 133.731 107.061) (end 133.731 108.331) (width 0.25) (layer B.Cu) (net 10))
+  (segment (start 133.731 108.331) (end 134.493 109.093) (width 0.25) (layer B.Cu) (net 10))
+  (segment (start 134.493 109.093) (end 146.304 109.093) (width 0.25) (layer B.Cu) (net 10))
   (segment (start 146.304 109.093) (end 147.701 107.696) (width 0.25) (layer B.Cu) (net 10))
-  (segment (start 134.493 109.093) (end 146.304 109.093) (width 0.25) (layer B.Cu) (net 10))
-  (segment (start 133.731 108.331) (end 134.493 109.093) (width 0.25) (layer B.Cu) (net 10))
-  (segment (start 133.731 107.061) (end 133.731 108.331) (width 0.25) (layer B.Cu) (net 10))
-  (segment (start 136.271 104.521) (end 133.731 107.061) (width 0.25) (layer B.Cu) (net 10))
   (segment (start 160.04 98.552) (end 156.337 98.552) (width 0.25) (layer F.Cu) (net 11))
   (segment (start 148.971 98.806) (end 147.701 100.076) (width 0.25) (layer F.Cu) (net 11))
@@
   (segment (start 156.337 98.552) (end 156.083 98.806) (width 0.25) (layer F.Cu) (net 11))
   (zone (net 12) (net_name "Net-(R1-Pad1)") (layer B.Cu) (hatch edge 0.508)
-    (connect_pads (clearance 0.508))
+    (connect_pads thru_hole_only (clearance 0.508))
     (min_thickness 0.254)
     (fill yes (arc_segments 16) (thermal_gap 0.508) (thermal_bridge_width 0.508))
