File: tower of power/tower of power.kicad_pcb (KiCad board)
At the start: 2 copper layers, 12 parts, among them J1 SerialIn, J2 SerialOut, SW1 SW_Push, SW2 SW_Push, SW3 SW_Push, U2 LEDStrip, U3 keypad

Commit message: finished tower maybe
Parts:
- removed DS1: WC1602A, Displays:WC1602A
- removed SW1, SW2: SW_Push, Buttons_Switches_THT:SW_PUSH_6mm_h4.3mm
- removed SW3: SW_Push, Buttons_Switches_THT:SW_PUSH-12mm
- added Advance1: SW_Push, Buttons_Switches_THT:SW_PUSH-12mm, F.Cu at (115.9, 105.7)
- added C1: C, Capacitors_THT:C_Disc_D5.0mm_W2.5mm_P5.00mm, B.Cu at (104.0, 98.2)
- added C2: C, Capacitors_THT:C_Disc_D5.0mm_W2.5mm_P5.00mm, B.Cu at (98.8, 98.2)
- added D1: D, Diodes_THT:D_A-405_P7.62mm_Horizontal, B.Cu at (50.3, 111.4)
- added J3: Conn_01x02, Pin_Headers:Pin_Header_Straight_1x02_Pitch2.54mm, B.Cu at (53.3, 116.4)
- added LCD1: WC1602A, Displays:WC1602A, F.Cu at (90.2, 28.8)
- added Q1: BC141, TO_SOT_Packages_THT:TO-92_Inline_Wide, B.Cu at (64.5, 116.5)
- added RN1: 10K, Resistors_THT:R_Array_SIP10, B.Cu at (55.2, 52.0)
- added Reset1: SW_Push, Buttons_Switches_THT:SW_PUSH_6mm_h4.3mm, B.Cu at (38.2, 106.4)
- added Return1: SW_Push, Buttons_Switches_THT:SW_PUSH-12mm, F.Cu at (74.0, 105.6)
- added SW4: Encoder, rocketlib:Encoder, F.Cu at (101.4, 83.4)
- A1, R1, RV1, U2: moved to B.Cu
- J1: value SerialIn -> Power; footprint Pin_Headers:Pin_Header_Straight_1x04_Pitch2.54mm -> Socket_Strips:Socket_Strip_Straight_1x02_Pitch2.54mm; moved to B.Cu
- J2: value SerialOut -> Serial; moved to B.Cu
- R2: footprint Resistors_THT:R_Axial_DIN0204_L3.6mm_D1.6mm_P5.08mm_Horizontal -> Resistors_THT:R_Axial_DIN0207_L6.3mm_D2.5mm_P7.62mm_Horizontal; moved to B.Cu
- moved R1 125.8 mm to (125.8, 31.8), turned to 270 degrees
- moved A1 113.0 mm to (36.4, 82.5), turned to 0 degrees
- moved U3 101.2 mm to (46.1, 95.0)
- moved U2 79.0 mm to (74.6, 57.8), turned to 270 degrees
- moved RV1 74.8 mm to (116.8, 40.5), turned to 90 degrees
- moved R2 53.2 mm to (60.7, 69.8), turned to 270 degrees
- moved J1 50.2 mm to (99.4, 115.9), turned to 270 degrees
- moved J2 34.4 mm to (34.6, 114.9), turned to 270 degrees
Connections:
- J1 pad 1: Net-(A1-Pad1) -> Vcc
- J1 pad 2: Net-(A1-Pad2) -> GND
- R2 pad 1: Vcc -> Net-(A1-Pad24)
- R2 pad 2: Net-(A1-Pad24) -> Net-(Q1-Pad2)
- U2 pad 1: Net-(A1-Pad23) -> Vcc
- U2 pad 2: GND -> Net-(A1-Pad23)
- U2 pad 3: (no net) -> GND
Routing:
- net Net-(A1-Pad10): track 0.00 -> 181.8 mm
- net Net-(A1-Pad21): track 0.00 -> 137.3 mm
- net Net-(A1-Pad6): track 0.00 -> 114.4 mm
- net Net-(A1-Pad19): track 0.00 -> 109.0 mm
- net Net-(A1-Pad11): track 0.00 -> 98.9 mm
- net Net-(A1-Pad5): track 0.00 -> 95.7 mm
- net Net-(A1-Pad12): track 0.00 -> 95.2 mm
- net Net-(A1-Pad13): track 0.00 -> 91.6 mm
- net Net-(A1-Pad14): track 0.00 -> 88.5 mm
- net Net-(A1-Pad22): track 0.00 -> 88.0 mm
- net Net-(A1-Pad15): track 0.00 -> 76.0 mm
- net Net-(A1-Pad16): track 0.00 -> 53.8 mm
- net Net-(LCD1-Pad3): track 0.00 -> 51.9 mm
- net Vcc: track 0.00 -> 50.1 mm
- net Net-(A1-Pad9): track 0.00 -> 42.9 mm
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- added copper zone on F.Cu, net GND
- added copper zone on B.Cu, net Vcc
Other:
- board outline added: 100 x 100 mm
