File: tower of power/tower of power.sch (KiCad schematic (older format))
At the start: 12 parts, among them J1 SerialIn, J2 SerialOut, SW1 SW_Push, SW2 SW_Push, SW3 SW_Push, SW4 Encoder, U2 LEDStrip, U3 keypad

Commit message: finished tower maybe
Parts:
- removed J1: SerialIn, Pin_Headers:Pin_Header_Straight_1x04_Pitch2.54mm, symbol Conn_01x04
- added C1, C2: C, Capacitors_THT:C_Disc_D5.0mm_W2.5mm_P5.00mm, symbol C
- added D1: D, Diodes_THT:D_A-405_P7.62mm_Horizontal, symbol D
- added J1: Power, Socket_Strips:Socket_Strip_Straight_1x02_Pitch2.54mm, symbol Conn_01x02
- added J3: Conn_01x02, Pin_Headers:Pin_Header_Straight_1x02_Pitch2.54mm, symbol Conn_01x02
- added Q1: BC141, TO_SOT_Packages_THT:TO-92_Inline_Wide, symbol BC141
- added R2: R, Resistors_THT:R_Axial_DIN0207_L6.3mm_D2.5mm_P7.62mm_Horizontal, symbol R
- added RN1: 10K, Resistors_THT:R_Array_SIP10, symbol R_Network09
- Advance1: renamed from SW2; footprint Buttons_Switches_THT:SW_PUSH_6mm_h4.3mm -> Buttons_Switches_THT:SW_PUSH-12mm
- J2: value SerialOut -> Serial
- SW4: footprint (none) -> rocketlib:Encoder
- renumbered DS1 to LCD1, SW1 to Reset1, SW3 to Return1
Connections:
- net GND: now also C1.1, C2.1, J1.2 (Pin_2), Q1.1 (E)
- net Vcc: now also D1.1 (K), J1.1 (Pin_1), J3.1 (Pin_1), RN1.1 (common)
- net at A1.19 (AD0/D14), U3.2 (R0): now also SW4.5, RN1.2 (R1); no longer SW4.4
- net at A1.20 (AD1/D15), U3.7 (R1): now also RN1.3 (R2)
- net at A1.21 (AD2/D16), U3.6 (R2): now also Advance1.2, RN1.4 (R3); no longer Advance1.1
- net at A1.22 (AD3/D17), U3.4 (R3): now also Return1.2, RN1.5 (R4); no longer Return1.1
- net at A1.24 (AD5/D19): now also R2.1
- net at A1.5 (D2), SW4.1 (A): now also C2.2, RN1.10 (R9)
- net at A1.6 (D3), SW4.3 (B): now also C1.2, RN1.9 (R8)
- new net: A1.10 (D7), Advance1.1, Return1.1, SW4.4
- new net: Q1.2 (B), R2.2
- new net: D1.2 (A), J3.2 (Pin_2), Q1.3 (C)
- no-connect marks 10 -> 12
Other:
- moved on the sheet: Advance1, Return1, SW4
