File: LED solder project/LED solder project.kicad_pcb (KiCad board)
At the start: 2 copper layers, 11 parts, among them Q1 PN2222A, SW1 SW_SPST

Commit message: update
Parts:
- SW1: footprint Buttons_Switches_THT:SW_DIP_x2_W7.62mm_Piano -> Pin_Headers:Pin_Header_Straight_1x03_Pitch2.54mm
- moved D3 65.6 mm to (163.8, 157.5), turned to 90 degrees
- moved D1 55.8 mm to (179.1, 157.5), turned to 90 degrees
- moved Q1 50.8 mm to (170.2, 138.4), turned to 90 degrees
- moved R2 49.9 mm to (157.5, 141.0), turned to 270 degrees
- moved D2 47.9 mm to (171.4, 157.5), turned to 90 degrees
- moved R3 41.4 mm to (179.1, 143.5), turned to 270 degrees
- moved R5 34.5 mm to (163.8, 143.5), turned to 270 degrees
- moved SW1 28.3 mm to (179.1, 130.8), turned to 90 degrees
- moved R1 24.8 mm to (157.5, 134.6), turned to 90 degrees
- moved R4 23.6 mm to (171.4, 143.5), turned to 270 degrees
- moved BT1 20.7 mm to (190.5, 138.4), turned to 270 degrees
Routing:
- net Net-(Q1-Pad3): track 0.00 -> 25.3 mm
- net Net-(Q1-Pad1): track 0.00 -> 20.8 mm
- net Net-(Q1-Pad2): track 0.00 -> 17.0 mm
- net VCC: track 0.00 -> 12.0 mm
- net Net-(D3-Pad2): track 0.00 -> 3.81 mm
- net Net-(D2-Pad2): track 0.00 -> 3.81 mm
- net Net-(D1-Pad2): track 0.00 -> 3.81 mm
- added copper zone on F.Cu, net GND

Commit message: added many
Parts:
- removed R1, R3, R4, R5: R, Resistors_THT:R_Axial_DIN0207_L6.3mm_D2.5mm_P7.62mm_Horizontal
- added 100: R, rocketlib:resistor, F.Cu at (133.3, 118.1)
- added 100: R, rocketlib:resistor, F.Cu at (128.9, 118.1)
- added 100: R, rocketlib:resistor, F.Cu at (137.8, 118.1)
- added 100: R, rocketlib:resistor, F.Cu at (142.9, 118.1)
- added 39K: R, rocketlib:resistor, F.Cu at (135.3, 110.5)
- added D4: LED, rocketlib:LED, F.Cu at (152.4, 134.6)
- BT1: footprint Pin_Headers:Pin_Header_Straight_2x01_Pitch2.54mm -> rocketlib:Battery
- D1, D2, D3: footprint LEDs:LED_D5.0mm -> rocketlib:LED
- Q1: footprint TO_SOT_Packages_THT:TO-92_Molded_Wide -> rocketlib:transistor
- R2: footprint Resistors_THT:R_Axial_DIN0414_L11.9mm_D4.5mm_P5.08mm_Vertical -> rocketlib:Photoresistor
- SW1: footprint Pin_Headers:Pin_Header_Straight_1x03_Pitch2.54mm -> rocketlib:Switch
- moved D1 46.6 mm to (138.4, 134.6), turned to 180 degrees
- moved D2 46.1 mm to (131.4, 134.6), turned to 180 degrees
- moved BT1 39.6 mm to (152.4, 127.6)
- moved R2 39.5 mm to (130.2, 112.4)
- moved SW1 32.1 mm to (152.4, 113.0), turned to 270 degrees
- moved D3 29.4 mm to (145.4, 134.6), turned to 180 degrees
- moved Q1 26.8 mm to (148.6, 122.6)
Routing:
- net Net-(Q1-Pad3): track 25.3 -> 0.00 mm
- net Net-(Q1-Pad1): track 20.8 -> 0.00 mm
- net Net-(Q1-Pad2): track 17.0 -> 0.00 mm
- net VCC: track 12.0 -> 0.00 mm
- net Net-(D3-Pad2): track 3.81 -> 0.00 mm
- net Net-(D2-Pad2): track 3.81 -> 0.00 mm
- net Net-(D1-Pad2): track 3.81 -> 0.00 mm
- removed copper zone on F.Cu, net GND
Other:
- board outline added: 27.2 x 29.8 mm

Commit message: updates
Connections:
- D4 pad 1: Net-(D4-Pad1) -> GND
Routing:
- net GND: track 0.00 -> 68.9 mm
- net Net-(Q1-Pad2): track 0.00 -> 22.6 mm
- net Net-(Q1-Pad1): track 0.00 -> 21.5 mm
- net VCC: track 0.00 -> 13.7 mm
- net Net-(Q1-Pad3): track 0.00 -> 11.7 mm
- net Net-(D4-Pad2): track 0.00 -> 8.56 mm
- net Net-(D3-Pad2): track 0.00 -> 6.66 mm
- net Net-(D1-Pad2): track 0.00 -> 4.86 mm
- net Net-(D2-Pad2): track 0.00 -> 3.81 mm
Other:
- board size 27.2 x 29.8 mm -> 27.9 x 30.4 mm
- board text added: "Designed by Collin Pearce"
Changed lines of the file:
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@@
 (kicad_pcb (version 4) (host pcbnew 4.0.7)
   (general
-    (links 17)
-    (no_connects 17)
-    (area 126.924999 107.874999 154.253001 137.870001)
+    (links 18)
+    (no_connects 0)
+    (area 126.162999 107.874999 154.253001 138.378001)
     (thickness 1.6)
-    (drawings 39)
-    (tracks 0)
+    (drawings 57)
+    (tracks 43)
     (zones 0)
     (modules 13)
-    (nets 11)
+    (nets 10)
   )
   (page A4)
   (layers
-    (0 F.Cu signal)
+    (0 F.Cu signal hide)
     (31 B.Cu signal)
     (32 B.Adhes user hide)
@@
     (34 B.Paste user hide)
     (35 F.Paste user hide)
-    (36 B.SilkS user hide)
-    (37 F.SilkS user)
+    (36 B.SilkS user)
+    (37 F.SilkS user hide)
     (38 B.Mask user hide)
     (39 F.Mask user hide)
@@
   (net 8 "Net-(Q1-Pad1)")
   (net 9 "Net-(D4-Pad2)")
-  (net 10 "Net-(D4-Pad1)")
   (net_class Default "This is the default net class."
     (clearance 0.2)
@@
     (add_net "Net-(D2-Pad2)")
     (add_net "Net-(D3-Pad2)")
-    (add_net "Net-(D4-Pad1)")
     (add_net "Net-(D4-Pad2)")
     (add_net "Net-(Q1-Pad1)")
@@
     )
     (pad 1 thru_hole rect (at 0 0 180) (size 1.8 1.8) (drill 0.9) (layers *.Cu *.Mask)
-      (net 10 "Net-(D4-Pad1)"))
+      (net 2 GND))
     (pad 2 thru_hole circle (at 2.54 0 180) (size 1.8 1.8) (drill 0.9) (layers *.Cu *.Mask)
       (net 9 "Net-(D4-Pad2)"))
@@
     )
   )
+  (gr_text "Designed by Collin Pearce" (at 141.605 114.3) (layer B.SilkS)
+    (effects (font (size 0.75 0.75) (thickness 0.1)) (justify mirror))
+  )
+  (gr_line (start 126.238 107.95) (end 127 107.95) (angle 90) (layer Edge.Cuts) (width 0.15))
+  (gr_line (start 126.238 108.077) (end 126.238 107.95) (angle 90) (layer Edge.Cuts) (width 0.15))
+  (gr_line (start 126.238 138.303) (end 127 138.303) (angle 90) (layer Edge.Cuts) (width 0.15))
+  (gr_line (start 126.238 137.922) (end 126.238 138.303) (angle 90) (layer Edge.Cuts) (width 0.15))
+  (gr_line (start 154.178 138.303) (end 154.178 137.795) (angle 90) (layer Edge.Cuts) (width 0.15))
+  (gr_line (start 133.35 134.62) (end 133.35 138.049) (angle 90) (layer F.SilkS) (width 0.1))
+  (gr_line (start 131.445 134.62) (end 133.35 134.62) (angle 90) (layer F.SilkS) (width 0.1))
+  (gr_line (start 140.335 134.62) (end 140.335 138.049) (angle 90) (layer F.SilkS) (width 0.1))
+  (gr_line (start 138.43 134.62) (end 140.335 134.62) (angle 90) (layer F.SilkS) (width 0.1))
+  (gr_line (start 147.32 134.62) (end 147.32 138.049) (angle 90) (layer F.SilkS) (width 0.1))
+  (gr_line (start 145.415 134.62) (end 147.32 134.62) (angle 90) (layer F.SilkS) (width 0.1))
+  (gr_line (start 152.4 134.62) (end 153.924 134.62) (angle 90) (layer F.SilkS) (width 0.1))
+  (gr_line (start 153.924 131.572) (end 153.924 138.049) (angle 90) (layer F.SilkS) (width 0.1))
+  (gr_line (start 152.4 130.048) (end 153.924 131.572) (angle 90) (layer F.SilkS) (width 0.1))
+  (gr_line (start 153.924 138.049) (end 126.619 138.049) (angle 90) (layer F.SilkS) (width 0.1))
+  (gr_line (start 126.619 118.364) (end 126.619 138.049) (angle 90) (layer F.SilkS) (width 0.1))
+  (gr_line (start 130.175 114.808) (end 126.619 118.364) (angle 90) (layer F.SilkS) (width 0.1))
+  (gr_line (start 134.366 109.982) (end 135.255 110.49) (angle 90) (layer F.SilkS) (width 0.1))
   (gr_line (start 133.35 132.08) (end 133.35 130.81) (angle 90) (layer F.SilkS) (width 0.1))
   (gr_line (start 135.89 134.62) (end 133.35 132.08) (angle 90) (layer F.SilkS) (width 0.1))
@@
   (gr_line (start 128.905 130.81) (end 128.905 134.62) (angle 90) (layer F.SilkS) (width 0.1))
   (gr_line (start 135.382 114.3) (end 135.255 114.3) (angle 90) (layer F.SilkS) (width 0.1))
-  (gr_line (start 148.59 120.015) (end 146.558 120.015) (angle 90) (layer F.SilkS) (width 0.1))
   (gr_line (start 128.905 118.11) (end 142.875 118.11) (angle 90) (layer F.SilkS) (width 0.1))
   (gr_line (start 150.241 110.49) (end 147.955 110.49) (angle 90) (layer F.SilkS) (width 0.1))
@@
   (gr_line (start 154.178 107.95) (end 127 107.95) (angle 90) (layer Edge.Cuts) (width 0.15))
   (gr_line (start 154.178 137.795) (end 154.178 107.95) (angle 90) (layer Edge.Cuts) (width 0.15))
-  (gr_line (start 127 137.795) (end 154.178 137.795) (angle 90) (layer Edge.Cuts) (width 0.15))
-  (gr_line (start 127 137.795) (end 127 107.95) (angle 90) (layer Edge.Cuts) (width 0.15))
+  (gr_line (start 127 138.303) (end 154.178 138.303) (angle 90) (layer Edge.Cuts) (width 0.15))
+  (gr_line (start 126.238 137.922) (end 126.238 108.077) (angle 90) (layer Edge.Cuts) (width 0.15))
+  (segment (start 152.4 125.095) (end 152.4 118.872) (width 0.25) (layer B.Cu) (net 1))
+  (segment (start 150.368 115.062) (end 152.4 113.03) (width 0.25) (layer B.Cu) (net 1))
+  (segment (start 150.368 116.84) (end 150.368 115.062) (width 0.25) (layer B.Cu) (net 1))
+  (segment (start 152.4 118.872) (end 150.368 116.84) (width 0.25) (layer B.Cu) (net 1))
+  (segment (start 138.43 134.62) (end 138.43 133.604) (width 0.25) (layer B.Cu) (net 2))
+  (segment (start 135.128 130.302) (end 135.128 127.635) (width 0.25) (layer B.Cu) (net 2))
+  (segment (start 138.43 133.604) (end 135.128 130.302) (width 0.25) (layer B.Cu) (net 2))
+  (segment (start 131.445 134.62) (end 131.445 128.397) (width 0.25) (layer B.Cu) (net 2))
+  (segment (start 131.445 128.397) (end 130.683 127.635) (width 0.25) (layer B.Cu) (net 2))
+  (segment (start 138.43 134.62) (end 138.43 134.366) (width 0.25) (layer B.Cu) (net 2))
+  (segment (start 145.415 134.62) (end 145.415 134.493) (width 0.25) (layer B.Cu) (net 2))
+  (segment (start 145.415 134.493) (end 143.51 132.588) (width 0.25) (layer B.Cu) (net 2))
+  (segment (start 143.51 132.588) (end 141.732 132.588) (width 0.25) (layer B.Cu) (net 2))
+  (segment (start 141.732 132.588) (end 140.589 131.445) (width 0.25) (layer B.Cu) (net 2))
+  (segment (start 140.589 131.445) (end 140.589 127.635) (width 0.25) (layer B.Cu) (net 2))
+  (segment (start 152.4 134.62) (end 152.4 130.048) (width 0.25) (layer B.Cu) (net 2))
+  (segment (start 130.175 114.808) (end 129.286 114.808) (width 0.25) (layer B.Cu) (net 2))
+  (segment (start 129.286 114.808) (end 127.635 116.459) (width 0.25) (layer B.Cu) (net 2))
+  (segment (start 127.635 116.459) (end 127.635 124.587) (width 0.25) (layer B.Cu) (net 2))
+  (segment (start 127.635 124.587) (end 130.683 127.635) (width 0.25) (layer B.Cu) (net 2))
+  (segment (start 130.683 127.635) (end 135.128 127.635) (width 0.25) (layer B.Cu) (net 2))
+  (segment (start 135.128 127.635) (end 140.589 127.635) (width 0.25) (layer B.Cu) (net 2))
+  (segment (start 140.589 127.635) (end 149.987 127.635) (width 0.25) (layer B.Cu) (net 2))
+  (segment (start 149.987 127.635) (end 152.4 130.048) (width 0.25) (layer B.Cu) (net 2))
+  (segment (start 135.89 134.62) (end 135.89 133.35) (width 0.25) (layer B.Cu) (net 3))
+  (segment (start 135.89 133.35) (end 133.35 130.81) (width 0.25) (layer B.Cu) (net 3))
+  (segment (start 128.905 134.62) (end 128.905 130.81) (width 0.25) (layer B.Cu) (net 4))
+  (segment (start 142.875 134.62) (end 141.605 134.62) (width 0.25) (layer B.Cu) (net 5))
+  (segment (start 141.605 134.62) (end 137.795 130.81) (width 0.25) (layer B.Cu) (net 5))
+  (segment (start 135.255 110.49) (end 139.065 110.49) (width 0.25) (layer B.Cu) (net 6))
+  (segment (start 139.065 110.49) (end 148.59 120.015) (width 0.25) (layer B.Cu) (net 6))
+  (segment (start 135.255 110.49) (end 130.683 110.49) (width 0.25) (layer B.Cu) (net 6))
+  (segment (start 130.683 110.49) (end 130.175 109.982) (width 0.25) (layer B.Cu) (net 6))
+  (segment (start 148.59 117.475) (end 148.59 111.125) (width 0.25) (layer B.Cu) (net 7))
+  (segment (start 148.59 111.125) (end 147.955 110.49) (width 0.25) (layer B.Cu) (net 7))
+  (segment (start 152.4 110.49) (end 147.955 110.49) (width 0.25) (layer B.Cu) (net 7))
+  (segment (start 128.905 118.11) (end 133.35 118.11) (width 0.25) (layer B.Cu) (net 8))
+  (segment (start 137.795 118.11) (end 133.35 118.11) (width 0.25) (layer B.Cu) (net 8))
+  (segment (start 142.875 118.11) (end 137.795 118.11) (width 0.25) (layer B.Cu) (net 8))
+  (segment (start 148.59 122.555) (end 147.32 122.555) (width 0.25) (layer B.Cu) (net 8))
+  (segment (start 147.32 122.555) (end 142.875 118.11) (width 0.25) (layer B.Cu) (net 8))
+  (segment (start 142.875 130.81) (end 146.05 130.81) (width 0.25) (layer B.Cu) (net 9))
+  (segment (start 146.05 130.81) (end 149.86 134.62) (width 0.25) (layer B.Cu) (net 9))
 )
